File: IICPP_Simul/DRG_Classic/EQ_Board/EQ_Board.kicad_sch (KiCad schematic)
At the start: 20 parts

Commit message: Reannotated Schems
Parts:
- renumbered C39 to C1, C40 to C2, C41 to C3, C42 to C4, C43 to C5, R63 to R1, R64 to R2, R65 to R3, R66 to R4, R67 to R5, RV9 to RV1, RV10 to RV2, RV11 to RV3, RV12 to RV4, RV13 to RV5
Changed lines of the file:
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@@
 		)
 	)
-	(text_box "TO DO\n----------------------------------------\nMake note of what is on board and what is not...\nAdd empty holes to go out for switches, pots, ground, etc.\nNeed 12AX7 Footprint.\nMake sure of trace width for signals, headters, VIAs, etc.\nLOOK MORE INTO ALL POT VALUES/TAPERS MORE\nResistors for heaters? Look into how heaters are usually AC run\nHow does the footswitch for eq, lead, and reverb work???\nSLAVE/DIRECT OUT? HOW DOES THIS TAP DIFFER FROM SEND?\n\nDONE\n----------------------------------------\nWHICH SIDE IS THE SWITCH ON FOR C++??\n-Mesa Mark III Schematic Says After C9\n\nFIND TAPER FOR RV5 (Lead Master)\n-General Consensus Says A, Consistent W/ Master 1\n\nLABEL ANODE/PLATE AND POWER RESISTOR WATTAGES\n-Generally 2W Metal Film, 3W if Labelled Otherwise\n-Anode/Plate Resistors are Part of Signal, Therefore Metal Film >> Metal Oxide"
+	(text_box "TO DO\n----------------------------------------\nMake note of what is on board and what is not...\nAdd empty holes to go out \nMake sure of trace width\n\nFilm or tant for caps?\nFind footprint for Mesa Sliders\nDo they use the minis?\n\nDONE\n----------------------------------------\n"
 		(exclude_from_sim no)
 		(at 195.58 55.88 0)
-		(size 64.77 53.34)
+		(size 64.77 35.56)
 		(margins 0.9525 0.9525 0.9525 0.9525)
 		(stroke
@@
 		(dnp no)
 		(fields_autoplaced yes)
-		(property "Reference" "R66"
+		(property "Reference" "R4"
 			(at 149.86 110.4899 0)
 			(effects
@@
 			(project "EQ_Board"
 				(path "/731158be-e106-4a86-bf06-392da2e983b4"
-					(reference "R66")
+					(reference "R4")
 					(unit 1)
 				)
@@
 		(dnp no)
 		(fields_autoplaced yes)
-		(property "Reference" "R63"
+		(property "Reference" "R1"
 			(at 101.6 110.4899 0)
 			(effects
@@
 			(project "EQ_Board"
 				(path "/731158be-e106-4a86-bf06-392da2e983b4"
-					(reference "R63")
+					(reference "R1")
 					(unit 1)
 				)
@@
 		(on_board yes)
 		(dnp no)
-		(property "Reference" "C42"
+		(property "Reference" "C4"
 			(at 151.13 131.6989 0)
 			(effects
@@
 			(project "EQ_Board"
 				(path "/731158be-e106-4a86-bf06-392da2e983b4"
-					(reference "C42")
+					(reference "C4")
 					(unit 1)
 				)
@@
 		(on_board yes)
 		(dnp no)
-		(property "Reference" "C43"
+		(property "Reference" "C5"
 			(at 167.64 131.6989 0)
 			(effects
@@
 			(project "EQ_Board"
 				(path "/731158be-e106-4a86-bf06-392da2e983b4"
-					(reference "C43")
+					(reference "C5")
 					(unit 1)
 				)
@@
 		(on_board yes)
 		(dnp no)
-		(property "Reference" "RV13"
+		(property "Reference" "RV5"
 			(at 156.21 97.7899 0)
 			(effects
@@
 			(project "EQ_Board"
 				(path "/731158be-e106-4a86-bf06-392da2e983b4"
-					(reference "RV13")
+					(reference "RV5")
 					(unit 1)
 				)
@@
 		(on_board yes)
 		(dnp no)
-		(property "Reference" "RV12"
+		(property "Reference" "RV4"
 			(at 139.7 97.7899 0)
 			(effects
@@
 			(project "EQ_Board"
 				(path "/731158be-e106-4a86-bf06-392da2e983b4"
-					(reference "RV12")
+					(reference "RV4")
 					(unit 1)
 				)
@@
 		(dnp no)
 		(fields_autoplaced yes)
-		(property "Reference" "R65"
+		(property "Reference" "R3"
 			(at 133.35 110.4899 0)
 			(effects
@@
 			(project "EQ_Board"
 				(path "/731158be-e106-4a86-bf06-392da2e983b4"
-					(reference "R65")
+					(reference "R3")
 					(unit 1)
 				)
@@
 		(on_board yes)
 		(dnp no)
-		(property "Reference" "C40"
+		(property "Reference" "C2"
 			(at 118.11 131.6989 0)
 			(effects
@@
 			(project "EQ_Board"
 				(path "/731158be-e106-4a86-bf06-392da2e983b4"
-					(reference "C40")
+					(reference "C2")
 					(unit 1)
 				)
@@
 		(on_board yes)
 		(dnp no)
-		(property "Reference" "RV9"
+		(property "Reference" "RV1"
 			(at 91.44 96.5199 0)
 			(effects
@@
 			(project "EQ_Board"
 				(path "/731158be-e106-4a86-bf06-392da2e983b4"
-					(reference "RV9")
+					(reference "RV1")
 					(unit 1)
 				)
@@
 		(on_board yes)
 		(dnp no)
-		(property "Reference" "RV10"
+		(property "Reference" "RV2"
 			(at 106.68 97.7899 0)
 			(effects
@@
 			(project "EQ_Board"
 				(path "/731158be-e106-4a86-bf06-392da2e983b4"
-					(reference "RV10")
+					(reference "RV2")
 					(unit 1)
 				)
@@
 		(dnp no)
 		(fields_autoplaced yes)
-		(property "Reference" "R67"
+		(property "Reference" "R5"
 			(at 166.37 110.4899 0)
 			(effects
@@
 			(project "EQ_Board"
 				(path "/731158be-e106-4a86-bf06-392da2e983b4"
-					(reference "R67")
+					(reference "R5")
 					(unit 1)
 				)
@@
 		(dnp no)
 		(fields_autoplaced yes)
-		(property "Reference" "R64"
+		(property "Reference" "R2"
 			(at 116.84 110.4899 0)
 			(effects
@@
 			(project "EQ_Board"
 				(path "/731158be-e106-4a86-bf06-392da2e983b4"
-					(reference "R64")
+					(reference "R2")
 					(unit 1)
 				)
@@
 		(on_board yes)
 		(dnp no)
-		(property "Reference" "C39"
+		(property "Reference" "C1"
 			(at 102.87 131.6989 0)
 			(effects
@@
 			(project "EQ_Board"
 				(path "/731158be-e106-4a86-bf06-392da2e983b4"
-					(reference "C39")
+					(reference "C1")
 					(unit 1)
 				)
@@
 		(on_board yes)
 		(dnp no)
-		(property "Reference" "C41"
+		(property "Reference" "C3"
 			(at 134.62 131.6989 0)
 			(effects
@@
 			(project "EQ_Board"
 				(path "/731158be-e106-4a86-bf06-392da2e983b4"
-					(reference "C41")
+					(reference "C3")
 					(unit 1)
 				)
@@
 		(on_board yes)
 		(dnp no)
-		(property "Reference" "RV11"
+		(property "Reference" "RV3"
 			(at 123.19 97.7899 0)
 			(effects
@@
 			(project "EQ_Board"
 				(path "/731158be-e106-4a86-bf06-392da2e983b4"
-					(reference "RV11")
+					(reference "RV3")
 					(unit 1)
 				)

Commit message: Added Annotations
Parts:
- L1: Notes (none) -> Mesa 519401
- L2: Notes (none) -> Mesa 519390
- L3: Notes (none) -> Mesa 519220
- L4: Notes (none) -> Mesa 519068
- L5: Notes (none) -> Mesa 519033
Changed lines of the file:
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@@
+	)
+	(junction
+		(at 93.98 144.78)
+		(diameter 0)
+		(color 0 0 0 0)
 	)
 	(junction
@@
 	)
 	(junction
-		(at 93.98 144.78)
-		(diameter 0)
-		(color 0 0 0 0)
-	)
-	(junction
 		(at 114.3 139.7)
 		(diameter 0)
@@
 	(wire
 		(pts
+			(xy 109.22 102.87) (xy 109.22 144.78)
+		)
+		(stroke
+			(width 0)
+			(type default)
+		)
+	)
+	(wire
+		(pts
+			(xy 142.24 144.78) (xy 158.75 144.78)
+		)
+		(stroke
+			(width 0)
+			(type default)
+		)
+	)
+	(wire
+		(pts
+			(xy 99.06 125.73) (xy 99.06 128.27)
+		)
+		(stroke
+			(width 0)
+			(type default)
+		)
+	)
+	(wire
+		(pts
+			(xy 109.22 90.17) (xy 109.22 95.25)
+		)
+		(stroke
+			(width 0)
+			(type default)
+		)
+	)
+	(wire
+		(pts
+			(xy 83.82 144.78) (xy 93.98 144.78)
+		)
+		(stroke
+			(width 0)
+			(type default)
+		)
+	)
+	(wire
+		(pts
 			(xy 93.98 144.78) (xy 109.22 144.78)
-		)
-		(stroke
-			(width 0)
-			(type default)
-		)
-	)
-	(wire
-		(pts
-			(xy 109.22 102.87) (xy 109.22 144.78)
-		)
-		(stroke
-			(width 0)
-			(type default)
-		)
-	)
-	(wire
-		(pts
-			(xy 142.24 144.78) (xy 158.75 144.78)
-		)
-		(stroke
-			(width 0)
-			(type default)
-		)
-	)
-	(wire
-		(pts
-			(xy 99.06 125.73) (xy 99.06 128.27)
-		)
-		(stroke
-			(width 0)
-			(type default)
-		)
-	)
-	(wire
-		(pts
-			(xy 109.22 90.17) (xy 109.22 95.25)
-		)
-		(stroke
-			(width 0)
-			(type default)
-		)
-	)
-	(wire
-		(pts
-			(xy 83.82 144.78) (xy 93.98 144.78)
 		)
 		(stroke
@@
 		(on_board yes)
 		(dnp no)
-		(fields_autoplaced yes)
 		(property "Reference" "L1"
 			(at 100.33 120.6499 0)
@@
 				)
 				(hide yes)
+			)
+		)
+		(property "Notes" "Mesa 519401"
+			(at 100.584 126.492 0)
+			(effects
+				(font
+					(size 1.27 1.27)
+				)
 			)
 		)
@@
 		(on_board yes)
 		(dnp no)
-		(fields_autoplaced yes)
 		(property "Reference" "L2"
 			(at 115.57 120.6499 0)
@@
 				)
 				(hide yes)
+			)
+		)
+		(property "Notes" "Mesa 519390"
+			(at 115.824 126.492 0)
+			(effects
+				(font
+					(size 1.27 1.27)
+				)
 			)
 		)
@@
 		(on_board yes)
 		(dnp no)
-		(fields_autoplaced yes)
 		(property "Reference" "L5"
 			(at 165.1 120.6499 0)
@@
 				)
 				(hide yes)
+			)
+		)
+		(property "Notes" "Mesa 519033"
+			(at 165.354 126.238 0)
+			(effects
+				(font
+					(size 1.27 1.27)
+				)
 			)
 		)
@@
 		(on_board yes)
 		(dnp no)
-		(fields_autoplaced yes)
 		(property "Reference" "L3"
 			(at 132.08 120.6499 0)
@@
 				)
 				(hide yes)
+			)
+		)
+		(property "Notes" "Mesa 519220"
+			(at 132.334 126.238 0)
+			(effects
+				(font
+					(size 1.27 1.27)
+				)
 			)
 		)
@@
 		(on_board yes)
 		(dnp no)
-		(fields_autoplaced yes)
 		(property "Reference" "L4"
 			(at 148.59 120.6499 0)
@@
 			)
 		)
+		(property "Notes" "Mesa 519068"
+			(at 148.844 126.238 0)
+			(effects
+				(font
+					(size 1.27 1.27)
+				)
+			)
+		)
