File: IICPP_Simul/DRG_Classic/EQ_Driver_Board/EQ_Driver_Board.kicad_sch (KiCad schematic)
At the start: 24 parts, among them Q1 MPSA63, Q2 MPSA70, Q3 MPSA70, Q4 MPSA20

Commit message: Reannotated Schems
Parts:
- renumbered C33 to C1, C34 to C2, C35 to C3, C44 to C4, C36 to C5, C37 to C6, C38 to C7, D7 to D1, R52 to R1, R60 to R10, R61 to R11, R62 to R12, R53 to R2, R54 to R3, R55 to R4, R56 to R5, R68 to R6, R57 to R7, R58 to R8, R59 to R9
Changed lines of the file:
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@@
 		)
 	)
-	(text_box "TO DO\n----------------------------------------\nMake note of what is on board and what is not...\nAdd empty holes to go out for switches, pots, ground, etc.\nNeed 12AX7 Footprint.\nMake sure of trace width for signals, headters, VIAs, etc.\nLOOK MORE INTO ALL POT VALUES/TAPERS MORE\nResistors for heaters? Look into how heaters are usually AC run\nHow does the footswitch for eq, lead, and reverb work???\nSLAVE/DIRECT OUT? HOW DOES THIS TAP DIFFER FROM SEND?\n\nDONE\n----------------------------------------\nWHICH SIDE IS THE SWITCH ON FOR C++??\n-Mesa Mark III Schematic Says After C9\n\nFIND TAPER FOR RV5 (Lead Master)\n-General Consensus Says A, Consistent W/ Master 1\n\nLABEL ANODE/PLATE AND POWER RESISTOR WATTAGES\n-Generally 2W Metal Film, 3W if Labelled Otherwise\n-Anode/Plate Resistors are Part of Signal, Therefore Metal Film >> Metal Oxide"
+	(text_box "TO DO\n----------------------------------------\nLook for transistor replacements\nLook for 100V and 63V footprints for Power Electros\nLook for Long and short 63V footprints for Other Electros\nAdd empty holes to go out\nMake sure of trace width\nFind out if 2W is appropriate for 470 and 220\n\nDONE\n----------------------------------------\n"
 		(exclude_from_sim no)
 		(at 199.39 88.9 0)
-		(size 64.77 53.34)
+		(size 64.77 33.02)
 		(margins 0.9525 0.9525 0.9525 0.9525)
 		(stroke
@@
 		(dnp no)
 		(fields_autoplaced yes)
-		(property "Reference" "R57"
+		(property "Reference" "R7"
 			(at 133.35 95.2499 0)
 			(effects
@@
 			(project "EQ_Driver_Board"
 				(path "/8b3e6737-4f8d-464d-ab54-70eaaf54bfcf"
-					(reference "R57")
+					(reference "R7")
 					(unit 1)
 				)
@@
 		(dnp no)
 		(fields_autoplaced yes)
-		(property "Reference" "R59"
+		(property "Reference" "R9"
 			(at 161.29 95.2499 0)
 			(effects
@@
 			(project "EQ_Driver_Board"
 				(path "/8b3e6737-4f8d-464d-ab54-70eaaf54bfcf"
-					(reference "R59")
+					(reference "R9")
 					(unit 1)
 				)
@@
 		(on_board yes)
 		(dnp no)
-		(property "Reference" "C36"
+		(property "Reference" "C5"
 			(at 164.719 74.93 90)
 			(effects
@@
 			(project "EQ_Driver_Board"
 				(path "/8b3e6737-4f8d-464d-ab54-70eaaf54bfcf"
-					(reference "C36")
+					(reference "C5")
 					(unit 1)
 				)
@@
 		(dnp no)
 		(fields_autoplaced yes)
-		(property "Reference" "R58"
+		(property "Reference" "R8"
 			(at 153.67 76.2 90)
 			(effects
@@
 			(project "EQ_Driver_Board"
 				(path "/8b3e6737-4f8d-464d-ab54-70eaaf54bfcf"
-					(reference "R58")
+					(reference "R8")
 					(unit 1)
 				)
@@
 		(dnp no)
 		(fields_autoplaced yes)
-		(property "Reference" "#PWR017"
+		(property "Reference" "#PWR03"
 			(at 191.77 82.55 0)
 			(effects
@@
 			(project "EQ_Driver_Board"
 				(path "/8b3e6737-4f8d-464d-ab54-70eaaf54bfcf"
-					(reference "#PWR017")
+					(reference "#PWR03")
 					(unit 1)
 				)
@@
 		(on_board yes)
 		(dnp no)
-		(property "Reference" "C34"
+		(property "Reference" "C2"
 			(at 77.47 74.93 90)
 			(effects
@@
 			(project "EQ_Driver_Board"
 				(path "/8b3e6737-4f8d-464d-ab54-70eaaf54bfcf"
-					(reference "C34")
+					(reference "C2")
 					(unit 1)
 				)
@@
 		(on_board yes)
 		(dnp no)
-		(property "Reference" "D7"
+		(property "Reference" "D1"
 			(at 210.82 52.07 0)
 			(effects
@@
 			(project "EQ_Driver_Board"
 				(path "/8b3e6737-4f8d-464d-ab54-70eaaf54bfcf"
-					(reference "D7")
+					(reference "D1")
 					(unit 1)
 				)
@@
 		(on_board yes)
 		(dnp no)
-		(property "Reference" "R68"
+		(property "Reference" "R6"
 			(at 109.22 93.98 90)
 			(effects
@@
 			(project "EQ_Driver_Board"
 				(path "/8b3e6737-4f8d-464d-ab54-70eaaf54bfcf"
-					(reference "R68")
+					(reference "R6")
 					(unit 1)
 				)
@@
 		(dnp no)
 		(fields_autoplaced yes)
-		(property "Reference" "R54"
+		(property "Reference" "R3"
 			(at 87.63 95.2499 0)
 			(effects
@@
 			(project "EQ_Driver_Board"
 				(path "/8b3e6737-4f8d-464d-ab54-70eaaf54bfcf"
-					(reference "R54")
+					(reference "R3")
 					(unit 1)
 				)
@@
 		(dnp no)
 		(fields_autoplaced yes)
-		(property "Reference" "R55"
+		(property "Reference" "R4"
 			(at 92.71 52.07 90)
 			(effects
@@
 			(project "EQ_Driver_Board"
 				(path "/8b3e6737-4f8d-464d-ab54-70eaaf54bfcf"
-					(reference "R55")
+					(reference "R4")
 					(unit 1)
 				)
@@
 		(on_board yes)
 		(dnp no)
-		(property "Reference" "C44"
+		(property "Reference" "C4"
 			(at 153.67 97.79 90)
 			(effects
@@
 			(project "EQ_Driver_Board"
 				(path "/8b3e6737-4f8d-464d-ab54-70eaaf54bfcf"
-					(reference "C44")
+					(reference "C4")
 					(unit 1)
 				)
@@
 		(on_board yes)
 		(dnp no)
-		(property "Reference" "R61"
+		(property "Reference" "R11"
 			(at 181.61 52.07 90)
 			(effects
@@
 			(project "EQ_Driver_Board"
 				(path "/8b3e6737-4f8d-464d-ab54-70eaaf54bfcf"
-					(reference "R61")
+					(reference "R11")
 					(unit 1)
 				)
@@
 		(dnp no)
 		(fields_autoplaced yes)
-		(property "Reference" "R52"
+		(property "Reference" "R1"
 			(at 73.66 95.2499 0)
 			(effects
@@
 			(project "EQ_Driver_Board"
 				(path "/8b3e6737-4f8d-464d-ab54-70eaaf54bfcf"
-					(reference "R52")
+					(reference "R1")
 					(unit 1)
 				)
@@
 		(dnp no)
 		(fields_autoplaced yes)
-		(property "Reference" "#PWR016"
+		(property "Reference" "#PWR02"
 			(at 158.75 106.68 0)
 			(effects
@@
 			(project "EQ_Driver_Board"
 				(path "/8b3e6737-4f8d-464d-ab54-70eaaf54bfcf"
-					(reference "#PWR016")
+					(reference "#PWR02")
 					(unit 1)
 				)
@@
 		(dnp no)
 		(fields_autoplaced yes)
-		(property "Reference" "R60"
+		(property "Reference" "R10"
 			(at 172.72 95.2499 0)
 			(effects
@@
 			(project "EQ_Driver_Board"
 				(path "/8b3e6737-4f8d-464d-ab54-70eaaf54bfcf"
-					(reference "R60")
+					(reference "R10")
 					(unit 1)
 				)
@@
 		(dnp no)
 		(fields_autoplaced yes)
-		(property "Reference" "#PWR015"
+		(property "Reference" "#PWR01"
 			(at 71.12 72.39 0)
 			(effects
@@
 			(project "EQ_Driver_Board"
 				(path "/8b3e6737-4f8d-464d-ab54-70eaaf54bfcf"
-					(reference "#PWR015")
+					(reference "#PWR01")
 					(unit 1)
 				)
@@
 		(dnp no)
 		(fields_autoplaced yes)
-		(property "Reference" "R56"
+		(property "Reference" "R5"
 			(at 101.6 95.2499 0)
 			(effects
@@
 			(project "EQ_Driver_Board"
 				(path "/8b3e6737-4f8d-464d-ab54-70eaaf54bfcf"
-					(reference "R56")
+					(reference "R5")
 					(unit 1)
 				)
@@
 		(on_board yes)
 		(dnp no)
-		(property "Reference" "C37"
+		(property "Reference" "C6"
 			(at 175.26 68.1989 0)
 			(effects
@@
 			(project "EQ_Driver_Board"
 				(path "/8b3e6737-4f8d-464d-ab54-70eaaf54bfcf"
-					(reference "C37")
+					(reference "C6")
 					(unit 1)
 				)
@@
 		(on_board yes)
 		(dnp no)
-		(property "Reference" "C35"
+		(property "Reference" "C3"
 			(at 148.59 64.77 90)
 			(effects
@@
 			(project "EQ_Driver_Board"
 				(path "/8b3e6737-4f8d-464d-ab54-70eaaf54bfcf"
-					(reference "C35")
+					(reference "C3")
 					(unit 1)
 				)
@@
 		(on_board yes)
 		(dnp no)
-		(property "Reference" "C38"
+		(property "Reference" "C7"
 			(at 195.58 68.1989 0)
 			(effects
@@
 			(project "EQ_Driver_Board"
 				(path "/8b3e6737-4f8d-464d-ab54-70eaaf54bfcf"
-					(reference "C38")
+					(reference "C7")
 					(unit 1)
 				)
@@
 		(dnp no)
 		(fields_autoplaced yes)
-		(property "Reference" "R53"
+		(property "Reference" "R2"
 			(at 87.63 68.5799 0)
 			(effects
@@
 			(project "EQ_Driver_Board"
 				(path "/8b3e6737-4f8d-464d-ab54-70eaaf54bfcf"
-					(reference "R53")
+					(reference "R2")
 					(unit 1)
 				)
@@
 		(on_board yes)
 		(dnp no)
-		(property "Reference" "R62"
+		(property "Reference" "R12"
 			(at 199.39 52.07 90)
 			(effects
@@
 			(project "EQ_Driver_Board"
 				(path "/8b3e6737-4f8d-464d-ab54-70eaaf54bfcf"
-					(reference "R62")
+					(reference "R12")
 					(unit 1)
 				)
@@
 		(on_board yes)
 		(dnp no)
-		(property "Reference" "C33"
+		(property "Reference" "C1"
 			(at 74.93 61.8489 0)
 			(effects
@@
 			(project "EQ_Driver_Board"
 				(path "/8b3e6737-4f8d-464d-ab54-70eaaf54bfcf"
-					(reference "C33")
+					(reference "C1")
 					(unit 1)
 				)

Commit message: Added Annotations
Other:
- note added: "C6 and C7 220uF are 63V on Original SLOCLONE uses 100V"
- note removed: "220uF are 63V on Original SLOCLONE uses 100V"
Changed lines of the file:
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@@
 	(generator_version "9.0")
 	(paper "A4")
-	(text "220uF are 63V on Original\nSLOCLONE uses 100V"
+	(text "C6 and C7 220uF are 63V on Original\nSLOCLONE uses 100V"
 		(exclude_from_sim no)
 		(at 181.356 46.99 0)
