File: IICPP_Simul/DRG_Classic/Preamp_Board/Preamp_Board.kicad_sch (KiCad schematic)
At the start: 121 parts, among them J1 Send, J2 Return, J3 Return, J4 Send, J5 Send, SW1 Pull Pot, SW2 Pull Pot, SW3 Pull Pot, SW4 Pull Pot, SW5 Pull Pot, SW6 Pull Pot, SW7 SW_SP3T, SW8 Pull Pot, SW9 Pull Pot, T1 Mesa 550185

Commit message: Reannotated Schems
Parts:
- renumbered C2 to C1, C16 to C10, C5 to C11, C9 to C12, C17 to C13, C1 to C15, C15 to C16, C10 to C17, C13 to C18, C31 to C19, C7 to C2, C29 to C22, C22 to C23, C26 to C24, C28 to C25, C19 to C26, C25 to C28, C23 to C29, C18 to C3, C24 to C30, C32 to C31, C30 to C32, C11 to C4, C12 to C5, C3 to C6, C8 to C7, C6 to C8, C4 to C9, D4 to D1, D5 to D3, D1 to D4, D3 to D5, R3 to R1, R14 to R11, R11 to R12, R1 to R13, R2 to R14, R4 to R15, R8 to R16, R9 to R17, R12 to R18, R7 to R2, R17 to R21, R18 to R22, R38 to R23, R39 to R24, R29 to R26, R33 to R27, R23 to R28, R28 to R29, R13 to R3, R35 to R30, R36 to R31, R37 to R32, R40 to R33, R41 to R34, R42 to R35, R24 to R36, R26 to R37, R27 to R38, R30 to R39, R21 to R4, R31 to R40, R32 to R41, R34 to R42, R44 to R43, R46 to R44, R51 to R45, R45 to R46, R48 to R47, R49 to R48, R50 to R49, R22 to R5, R43 to R50, R47 to R51, R15 to R6, R6 to R7, R16 to R8, R5 to R9, RV6 to RV2, RV2 to RV3, RV5 to RV4, RV4 to RV5, RV3 to RV6, RV8 to RV7, RV7 to RV8, SW2 to SW1, SW3 to SW2, SW4 to SW3, SW1 to SW4, V4 to V3, V3 to V4

Commit message: Added Annotations
Other:
- note added: "C10, SW3 for C++"
- note added: "C25 Unknown Voltage Assumed to be Consistent W/ Other T322 Cathode Bypass Caps"
- note added: "R12, C12, SW2 for C++"
- note added: "R36 Hardwired for C++"
- note added: "R5 Potentially Optional? Used to even out Master 1 Taper"
- note added: "Remove C19 on Simul"
- note added: "Remove C30 on Simul (SLOCLONE) Keep C30 on Simul (JRB32)"
- note removed: "C28 Unknown Voltage Assumed to be Consistent W/ Other T322 Cathode Bypass Caps"
- note removed: "R22 Potentially Optional? Used to even out Master 1 Taper"
- note removed: "R24 Hardwired for C++"
- note removed: "Remove C24 on Simul (SLOCLONE) Keep C24 on Simul (JRB32)"
- note removed: "Remove C31 on Simul"
Changed lines of the file:
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@@
 		)
 	)
-	(text "C28 Unknown Voltage\nAssumed to be Consistent W/ Other T322 Cathode Bypass Caps"
+	(text "C25 Unknown Voltage\nAssumed to be Consistent W/ Other T322 Cathode Bypass Caps"
 		(exclude_from_sim no)
 		(at 396.494 230.124 0)
+		(effects
+			(font
+				(size 1.27 1.27)
+			)
+		)
+	)
+	(text "C10, SW3 for C++"
+		(exclude_from_sim no)
+		(at 285.496 131.572 0)
 		(effects
 			(font
@@
 		)
 	)
-	(text "R24 Hardwired for C++"
+	(text "R36 Hardwired for C++"
 		(exclude_from_sim no)
 		(at 123.952 231.394 0)
@@
 		)
 	)
-	(text "Remove C24 on Simul (SLOCLONE)\nKeep C24 on Simul (JRB32)\n"
+	(text "Remove C30 on Simul (SLOCLONE)\nKeep C30 on Simul (JRB32)\n"
 		(exclude_from_sim no)
 		(at 238.76 232.156 0)
@@
 		)
 	)
-	(text "R22 Potentially Optional?\nUsed to even out Master 1 Taper"
+	(text "R5 Potentially Optional?\nUsed to even out Master 1 Taper"
 		(exclude_from_sim no)
 		(at 405.892 55.372 0)
@@
 		)
 	)
-	(text "Remove C31 on Simul"
+	(text "Remove C19 on Simul"
 		(exclude_from_sim no)
 		(at 201.93 159.512 0)
 		(effects
 			(font
+				(size 1.27 1.27)
+			)
+		)
+	)
+	(text "R12, C12, SW2 for C++"
+		(exclude_from_sim no)
+		(at 248.158 111.76 0)
+		(effects
+			(font
