File: Classic_Preamp_Board_R_EQ/Classic_Preamp_Board_R_EQ.kicad_sch (KiCad schematic)
At the start: 121 parts, among them J1 Send, J2 Return, J3 Return, J4 Send, J5 Send, SW1 Pull Pot, SW2 Pull Pot, SW3 Pull Pot, SW4 Pull Pot, SW5 Pull Pot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

Commit message: Updated Schematics and Organizational Structure
Parts:
- removed R47: 470, symbol Device:R
- added R45: 68K, symbol Device:R
- LDR4, LDR5: value VTL5C4 -> NSL-32SR2
- R43: value 220 -> 680
- R44: value 470 -> 220
- R46: value 680 -> 470
- R47: renamed from R45; Notes 3W Metal Oxide -> 2W Metal Oxide
- R48: value 100 -> 680; Notes (none) -> 3W Wirewound
- R49: value 68K -> 3K3
- R50: value 680 -> 100; Notes 3W Wirewound -> (none)
- R51: value 3K3 -> 470
- renumbered D2 to D1, D3 to D2, D1 to D3
Connections:
- net GEQ: now also R45.1; no longer R49.1
- net GND: now also R44.2, R45.2; no longer R43.1, R49.2
- net LDR2-: now also R49.2, R50.1; no longer R48.1
- net at J5.T: now also R50.2; no longer R48.2
- net at C32.1, D5.1 (K), R51.1: now also R43.1, R48.2, R49.1; no longer R46.1, R50.2
- net at D4.1 (K): now also R48.1; no longer R50.1
- net at LDR5.1 (-), SW7.3: now also R46.1; no longer R44.1
- net at D2.2 (A): now also R46.2; no longer R44.2
- net at SW7.1: now also R44.1; no longer R43.2
- net at D1.1 (K), LDR5.2 (+): now also R43.2; no longer R46.2
Other:
- note added: "EQ Footswitch Overrides All Modes"
- note added: "EQ IN: EQ Always Engaged EQ OUT: EQ Off EQ AUTO: EQ Engaged W/ Lead"
- note added: "Original: VTL5C4"
- note added: "Treble Shift Only Works W/ Lead Engaged"
- moved on the sheet: D1, D2, D3, D4, D5, D6, J5, LDR5, R13, SW8, SW9, V3C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
