File: EQ Boards/EQ_Driver_Board/EQ_Driver_Board.kicad_pcb (KiCad board)
At the start: 2 copper layers, 127 x 57.2 mm, 34 parts, among them Q1 MPSA63, Q2 MPSA70, Q3 MPSA70, Q4 MPSA20

Commit message: EQ Slider Board Progress
Other:
- board text added: "HCF EQ DRIVER"
- board text removed: "HCF IIC++ EQ DRIVER"
Changed lines of the file:
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@@
 		)
 		(property "Value" "Power"
-			(at 0 1 0)
+			(at 0.12 -2.86 0)
 			(unlocked yes)
-			(layer "F.Fab")
-			(hide yes)
+			(layer "F.SilkS")
 			(effects
 				(font
@@
 		)
 		(property "Value" "EQ Input"
-			(at 0 1 0)
+			(at -0.05 3.025 0)
 			(unlocked yes)
-			(layer "F.Fab")
-			(hide yes)
+			(layer "F.SilkS")
 			(effects
 				(font
@@
 		)
 		(property "Value" "GND"
-			(at 0 1 0)
+			(at 0.02 3.02 0)
 			(unlocked yes)
-			(layer "F.Fab")
-			(hide yes)
+			(layer "F.SilkS")
 			(effects
 				(font
@@
 		)
 		(property "Value" "Cut (L)"
-			(at 0 1 0)
+			(at 0 -3.07 0)
 			(unlocked yes)
-			(layer "F.Fab")
-			(hide yes)
+			(layer "F.SilkS")
 			(effects
 				(font
@@
 		)
 		(property "Value" "Boost (R)"
-			(at 0 1 0)
+			(at 0 -3.02 0)
 			(unlocked yes)
-			(layer "F.Fab")
-			(hide yes)
+			(layer "F.SilkS")
 			(effects
 				(font
@@
 		)
 	)
-	(gr_text "HCF IIC++\nEQ DRIVER"
-		(at 174.4472 118.11 0)
+	(gr_text "HCF\nEQ DRIVER"
+		(at 180.22 117.82 0)
 		(layer "F.SilkS")
 		(effects
@@
 				(bold yes)
 			)
-			(justify left bottom)
+			(justify bottom)
 		)
 	)
