File: EQ Boards/EQ_Slider_Board/EQ_Slider_Board.kicad_pcb (KiCad board)
At the start: 2 copper layers, 11 parts

Commit message: EQ Slider Board Progress
Parts:
- added C5: 0.033uF, Capacitor_THT:C_Rect_L7.2mm_W2.5mm_P5.00mm_FKS2_FKP2_MKS2_MKP2, F.Cu at (115.5, 82.2)
- added L1: 1.0H, HiroFootprints:MB Inductor, F.Cu at (177.0, 104.8)
- added L2: 0.39H, HiroFootprints:MB Inductor, F.Cu at (161.6, 104.8)
- added L3: 0.22H, HiroFootprints:MB Inductor, F.Cu at (146.2, 104.8)
- added L4: 0.068H, HiroFootprints:MB Inductor, F.Cu at (130.8, 104.8)
- added L5: 0.033H, HiroFootprints:MB Inductor, F.Cu at (115.5, 104.8)
- added REF**: MountingHole_4mm, MountingHole:MountingHole_4mm, F.Cu at (211.3, 125.7)
- added REF**: MountingHole_4mm, MountingHole:MountingHole_4mm, F.Cu at (108.2, 70.8)
- added REF**: MountingHole_4mm, MountingHole:MountingHole_4mm, F.Cu at (211.3, 70.8)
- added REF**: MountingHole_4mm, MountingHole:MountingHole_4mm, F.Cu at (108.2, 125.7)
- added RV1: 50K, HiroFootprints:Mesa 588536, B.Cu at (188.2, 124.0)
- added RV2: 50K, HiroFootprints:Mesa 588536, B.Cu at (172.8, 124.0)
- added RV3: 50K, HiroFootprints:Mesa 588536, B.Cu at (157.4, 124.0)
- added RV4: 50K, HiroFootprints:Mesa 588536, B.Cu at (142.0, 124.0)
- added RV5: 50K, HiroFootprints:Mesa 588536, B.Cu at (126.6, 124.0)
- TP3: value GEQ -> GEQ LDR
- moved TP1 66.9 mm to (198.2, 110.8)
- moved R1 63.2 mm to (177.0, 123.3), turned to 90 degrees
- moved C3 49.1 mm to (146.9, 71.0), turned to -90 degrees
- moved TP2 46.2 mm to (198.2, 98.5)
- moved R2 45.5 mm to (161.6, 123.3), turned to 90 degrees
- moved R3 28.9 mm to (146.2, 123.3), turned to 90 degrees
- moved C2 25.8 mm to (162.3, 71.1), turned to -90 degrees
- moved C1 16.2 mm to (177.7, 71.0), turned to -90 degrees
- moved TP3 12.7 mm to (206.8, 98.5)
- moved R4 11.8 mm to (130.8, 123.3), turned to 90 degrees
- moved R5 5.61 mm to (115.5, 123.3), turned to 90 degrees
Routing:
- net Net-(RV1-Pad3): track 0.00 -> 127.8 mm
- net Net-(RV1-Pad1): track 0.00 -> 72.9 mm
- net Net-(R5-Pad1): track 0.00 -> 13.1 mm
- net Net-(R1-Pad1): track 0.00 -> 13.1 mm
- net Net-(R2-Pad1): track 0.00 -> 13.1 mm
- net Net-(R4-Pad1): track 0.00 -> 13.1 mm
- net Net-(R3-Pad1): track 0.00 -> 13.1 mm
- net Net-(C5-Pad2): track 0.00 -> 4.89 mm
- net Net-(L3-Pad1): track 0.00 -> 3.25 mm
- net Net-(L5-Pad1): track 0.00 -> 3.25 mm
- net Net-(L4-Pad1): track 0.00 -> 3.25 mm
- net Net-(L2-Pad1): track 0.00 -> 3.25 mm
- net Net-(L1-Pad1): track 0.00 -> 3.25 mm
Other:
- board outline added: 111.8 x 63.5 mm
- board text added: "HCF EQ Slider"
- board text added: "Ver 1.0"

Commit message: Finished EQ Slider V1 Board
Parts:
- added C4: 0.15uF, Capacitor_THT:CP_Radial_Tantal_D4.5mm_P5.00mm, F.Cu at (131.3, 75.8)
- moved TP3 29.7 mm to (195.8, 70.8)
- moved TP1 22.7 mm to (195.8, 88.2)
- moved TP2 20.4 mm to (195.8, 78.2)
- moved REF** 8.53 mm to (202.8, 71.2)
- moved REF** 8.53 mm to (202.8, 126.0)
- moved REF** 1.69 mm to (109.8, 71.2)
- moved REF** 1.68 mm to (109.8, 126.0)
- moved C2 0.31 mm to (162.4, 70.8)
- moved C3 0.29 mm to (147.1, 70.8)
- moved C1 0.25 mm to (177.6, 70.8)
Routing:
- net Net-(C1-Pad1): track 0.00 -> 92.2 mm
- net Net-(RV1-Pad3): track 127.8 -> 148.7 mm
- net Net-(C4-Pad2): track 0.00 -> 11.5 mm
- net Net-(C3-Pad2): track 0.00 -> 6.65 mm
- net Net-(C2-Pad2): track 0.00 -> 6.64 mm
- net Net-(RV1-Pad1): track 72.9 -> 69.2 mm
- net Net-(C1-Pad2): track 0.00 -> 3.53 mm
Other:
- board size 111.8 x 63.5 mm -> 101.6 x 63.5 mm
