File: EQ Boards/EQ_Slider_Board/EQ_Slider_Board.kicad_sch (KiCad schematic)
At the start: 20 parts

Commit message: Updated Schematics and Organizational Structure
Parts:
- added TP1: Cut (L), HiroFootprints:Out_Hole_3.4_1.8, symbol Connector:TestPoint
- added TP2: Boost (R), HiroFootprints:Out_Hole_3.4_1.8, symbol Connector:TestPoint
- added TP3: GEQ, HiroFootprints:Out_Hole_3.4_1.8, symbol Connector:TestPoint
- C1: footprint (none) -> Capacitor_THT:CP_Axial_L11.0mm_D5.0mm_P18.00mm_Horizontal
- C2, C3: footprint (none) -> Capacitor_THT:CP_Axial_L10.0mm_D4.5mm_P15.00mm_Horizontal
- R1, R2, R3, R4, R5: footprint (none) -> Resistor_THT:R_Axial_DIN0411_L9.9mm_D3.6mm_P15.24mm_Horizontal
Connections:
- net EQ Left: no longer names the net of RV1.3, RV2.3, RV3.3, RV4.3, RV5.3
- net EQ Left: now also TP1.1
- net EQ Right: no longer names the net of RV1.1, RV2.1, RV3.1, RV4.1, RV5.1
- net EQ Right: now also TP2.1
- net GEQ: no longer names the net of C1.1, C2.1, C3.1, C4.1, C5.1
- net GEQ: now also TP3.1
Changed lines of the file:
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@@
 		)
 	)
-	(text_box "TO DO\n----------------------------------------\nMake note of what is on board and what is not...\nAdd empty holes to go out \nMake sure of trace width\n\nFilm or tant for caps?\nFind footprint for Mesa Sliders\nDo they use the minis?\n\nDONE\n----------------------------------------\n"
-		(exclude_from_sim no)
-		(at 195.58 55.88 0)
+	(text_box "TO DO\n----------------------------------------\nMake note of what is on board and what is not...\n\n\n\nFind footprint for Mesa Sliders\n\n\nDONE\n----------------------------------------\n"
+		(exclude_from_sim no)
+		(at 187.96 73.66 0)
 		(size 64.77 35.56)
 		(margins 0.9525 0.9525 0.9525 0.9525)
@@
 		)
 	)
-	(text_box "EQ"
+	(text_box "EQ Slider"
 		(exclude_from_sim no)
 		(at 71.12 68.58 0)
@@
 	(wire
 		(pts
-			(xy 163.83 139.7) (xy 170.18 139.7)
+			(xy 163.83 139.7) (xy 172.72 139.7)
 		)
 		(stroke
@@
 			(width 0)
 			(type default)
-		)
-	)
-	(global_label "GEQ"
-		(shape output)
-		(at 170.18 139.7 0)
-		(fields_autoplaced yes)
-		(effects
-			(font
-				(size 1.27 1.27)
-			)
-			(justify left)
-		)
-		(property "Intersheetrefs" "${INTERSHEET_REFS}"
-			(at 176.9147 139.7 0)
-			(effects
-				(font
-					(size 1.27 1.27)
-				)
-				(justify left)
-				(hide yes)
-			)
-		)
-	)
-	(global_label "EQ Left"
-		(shape output)
-		(at 125.73 72.39 90)
-		(fields_autoplaced yes)
-		(effects
-			(font
-				(size 1.27 1.27)
-			)
-			(justify left)
-		)
-		(property "Intersheetrefs" "${INTERSHEET_REFS}"
-			(at 125.73 62.3896 90)
-			(effects
-				(font
-					(size 1.27 1.27)
-				)
-				(justify left)
-				(hide yes)
-			)
-		)
-	)
-	(global_label "EQ Right"
-		(shape output)
-		(at 158.75 72.39 90)
-		(fields_autoplaced yes)
-		(effects
-			(font
-				(size 1.27 1.27)
-			)
-			(justify left)
-		)
-		(property "Intersheetrefs" "${INTERSHEET_REFS}"
-			(at 158.75 61.0592 90)
-			(effects
-				(font
-					(size 1.27 1.27)
-				)
-				(justify left)
-				(hide yes)
-			)
 		)
 	)
@@
 			)
 		)
-		(property "Footprint" ""
+		(property "Footprint" "Resistor_THT:R_Axial_DIN0411_L9.9mm_D3.6mm_P15.24mm_Horizontal"
 			(at 145.542 111.76 90)
 			(effects
@@
 			)
 		)
-		(property "Footprint" ""
+		(property "Footprint" "Resistor_THT:R_Axial_DIN0411_L9.9mm_D3.6mm_P15.24mm_Horizontal"
 			(at 97.282 111.76 90)
 			(effects
@@
 				(path "/731158be-e106-4a86-bf06-392da2e983b4"
 					(reference "C4")
+					(unit 1)
+				)
+			)
+		)
+	)
+	(symbol
+		(lib_id "Connector:TestPoint")
+		(at 172.72 139.7 270)
+		(unit 1)
+		(exclude_from_sim no)
+		(in_bom yes)
+		(on_board yes)
+		(dnp no)
+		(fields_autoplaced yes)
+		(property "Reference" "TP3"
+			(at 177.8 138.4299 90)
+			(effects
+				(font
+					(size 1.27 1.27)
+				)
+				(justify left)
+			)
+		)
+		(property "Value" "GEQ"
+			(at 177.8 140.9699 90)
+			(effects
+				(font
+					(size 1.27 1.27)
+				)
+				(justify left)
+			)
+		)
+		(property "Footprint" "HiroFootprints:Out_Hole_3.4_1.8"
+			(at 172.72 144.78 0)
+			(effects
+				(font
+					(size 1.27 1.27)
+				)
+				(hide yes)
+			)
+		)
+		(property "Datasheet" "~"
+			(at 172.72 144.78 0)
+			(effects
+				(font
+					(size 1.27 1.27)
+				)
+				(hide yes)
+			)
+		)
+		(property "Description" "test point"
+			(at 172.72 139.7 0)
+			(effects
+				(font
+					(size 1.27 1.27)
+				)
+				(hide yes)
+			)
+		)
+		(pin "1"
+		)
+		(instances
+			(project "EQ_Slider_Board"
+				(path "/731158be-e106-4a86-bf06-392da2e983b4"
+					(reference "TP3")
 					(unit 1)
 				)
@@
 			)
 		)
-		(property "Footprint" ""
+		(property "Footprint" "Resistor_THT:R_Axial_DIN0411_L9.9mm_D3.6mm_P15.24mm_Horizontal"
 			(at 129.032 111.76 90)
 			(effects
@@
 			)
 		)
-		(property "Footprint" ""
+		(property "Footprint" "Capacitor_THT:CP_Axial_L10.0mm_D4.5mm_P15.00mm_Horizontal"
 			(at 113.3348 128.27 0)
 			(effects
@@
 			)
 		)
-		(property "Footprint" ""
+		(property "Footprint" "Resistor_THT:R_Axial_DIN0411_L9.9mm_D3.6mm_P15.24mm_Horizontal"
 			(at 162.052 111.76 90)
 			(effects
@@
 			)
 		)
-		(property "Footprint" ""
+		(property "Footprint" "Resistor_THT:R_Axial_DIN0411_L9.9mm_D3.6mm_P15.24mm_Horizontal"
 			(at 112.522 111.76 90)
 			(effects
@@
 			)
 		)
-		(property "Footprint" ""
+		(property "Footprint" "Capacitor_THT:CP_Axial_L11.0mm_D5.0mm_P18.00mm_Horizontal"
 			(at 98.0948 128.27 0)
 			(effects
@@
 			)
 		)
-		(property "Footprint" ""
+		(property "Footprint" "Capacitor_THT:CP_Axial_L10.0mm_D4.5mm_P15.00mm_Horizontal"
 			(at 129.8448 128.27 0)
 			(effects
@@
 					(unit 1)
 				)
+			)
+		)
+	)
+	(symbol
+		(lib_id "Connector:TestPoint")
+		(at 125.73 72.39 0)
+		(unit 1)
+		(exclude_from_sim no)
+		(in_bom yes)
+		(on_board yes)
+		(dnp no)
+		(fields_autoplaced yes)
+		(property "Reference" "TP1"
+			(at 128.27 67.8179 0)
+			(effects
+				(font
+					(size 1.27 1.27)
+				)
+				(justify left)
+			)
+		)
+		(property "Value" "Cut (L)"
+			(at 128.27 70.3579 0)
+			(effects
+				(font
+					(size 1.27 1.27)
+				)
+				(justify left)
+			)
+		)
+		(property "Footprint" "HiroFootprints:Out_Hole_3.4_1.8"
+			(at 130.81 72.39 0)
+			(effects
+				(font
+					(size 1.27 1.27)
+				)
+				(hide yes)
+			)
+		)
+		(property "Datasheet" "~"
+			(at 130.81 72.39 0)
+			(effects
+				(font
+					(size 1.27 1.27)
+				)
+				(hide yes)
+			)
+		)
+		(property "Description" "test point"
+			(at 125.73 72.39 0)
+			(effects
+				(font
+					(size 1.27 1.27)
+				)
+				(hide yes)
+			)
+		)
+		(pin "1"
+		)
+		(instances
+			(project ""
+				(path "/731158be-e106-4a86-bf06-392da2e983b4"
+					(reference "TP1")
+					(unit 1)
+				)
+			)
+		)
+	)
+	(symbol
+		(lib_id "Connector:TestPoint")
+		(at 158.75 72.39 0)
+		(unit 1)
+		(exclude_from_sim no)
+		(in_bom yes)
+		(on_board yes)
+		(dnp no)
+		(fields_autoplaced yes)
+		(property "Reference" "TP2"
+			(at 161.29 67.8179 0)
+			(effects
+				(font
+					(size 1.27 1.27)
+				)
+				(justify left)
+			)
+		)
+		(property "Value" "Boost (R)"
+			(at 161.29 70.3579 0)
+			(effects
+				(font
+					(size 1.27 1.27)
+				)
+				(justify left)
+			)
+		)
+		(property "Footprint" "HiroFootprints:Out_Hole_3.4_1.8"
+			(at 163.83 72.39 0)
+			(effects
+				(font
+					(size 1.27 1.27)
+				)
+				(hide yes)
+			)
+		)
+		(property "Datasheet" "~"
+			(at 163.83 72.39 0)
+			(effects
+				(font
+					(size 1.27 1.27)
+				)
+				(hide yes)
+			)
+		)
+		(property "Description" "test point"
+			(at 158.75 72.39 0)
+			(effects
+				(font
+					(size 1.27 1.27)
+				)
+				(hide yes)
+			)
+		)
+		(pin "1"
+		)
+		(instances
+			(project "EQ_Slider_Board"
+				(path "/731158be-e106-4a86-bf06-392da2e983b4"
+					(reference "TP2")
+					(unit 1)
+				)

Commit message: EQ Slider Board Progress
Parts:
- C5: footprint (none) -> Capacitor_THT:C_Rect_L7.2mm_W2.5mm_P5.00mm_FKS2_FKP2_MKS2_MKP2
- L1, L2, L3, L4, L5: footprint (none) -> HiroFootprints:MB Inductor
- RV1, RV2, RV3, RV4, RV5: footprint (none) -> HiroFootprints:Mesa 588536
- TP3: value GEQ -> GEQ LDR
Other:
- note added: "C1, C2, C3: T322 Used"
- note added: "C4: T356 Used T110, and Film Caps Available As Well"
- note added: "C5: 0.033uF 50V Film Cap Used Instead"
Changed lines of the file:
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@@
 	(generator_version "9.0")
 	(paper "A4")
+	(text "C5: 0.033uF 50V Film Cap \nUsed Instead"
+		(exclude_from_sim no)
+		(at 185.674 132.08 0)
+		(effects
+			(font
+				(size 1.27 1.27)
+			)
+		)
+	)
+	(text "C4: T356 Used\nT110, and Film Caps\nAvailable As Well"
+		(exclude_from_sim no)
+		(at 150.876 150.114 0)
+		(effects
+			(font
+				(size 1.27 1.27)
+			)
+		)
+	)
+	(text "C1, C2, C3: T322 Used"
+		(exclude_from_sim no)
+		(at 115.062 148.844 0)
+		(effects
+			(font
+				(size 1.27 1.27)
+			)
+		)
+	)
 	(text_box "ALL RESISTORS ARE 1W METAL FILM UNLESS LABELLED OTHERWISE\nCAP VOLTAGES AND MODELS ARE SPECIFIC TO MY BUILD\nSCHEMATIC MODELED AFTER SLOCLONE, DANO, JAY OMEGA, AND JRB32 VERSIONS"
 		(exclude_from_sim no)
@@
 		)
 	)
-	(text_box "TO DO\n----------------------------------------\nMake note of what is on board and what is not...\n\n\n\nFind footprint for Mesa Sliders\n\n\nDONE\n----------------------------------------\n"
+	(text_box "TO DO\n----------------------------------------\nMake note of what is on board and what is not...\n\nFind boost and cut filter points\n\n\nDONE\n----------------------------------------\n"
 		(exclude_from_sim no)
 		(at 187.96 73.66 0)
@@
 			)
 		)
-		(property "Footprint" ""
+		(property "Footprint" "HiroFootprints:MB Inductor"
 			(at 99.06 121.92 0)
 			(effects
@@
 			)
 		)
-		(property "Footprint" ""
+		(property "Footprint" "HiroFootprints:MB Inductor"
 			(at 114.3 121.92 0)
 			(effects
@@
 			)
 		)
-		(property "Value" "GEQ"
+		(property "Value" "GEQ LDR"
 			(at 177.8 140.9699 90)
 			(effects
@@
 			)
 		)
-		(property "Footprint" ""
+		(property "Footprint" "Capacitor_THT:C_Rect_L7.2mm_W2.5mm_P5.00mm_FKS2_FKP2_MKS2_MKP2"
 			(at 162.8648 128.27 0)
 			(effects
@@
 			)
 		)
-		(property "Footprint" ""
+		(property "Footprint" "HiroFootprints:Mesa 588536"
 			(at 158.75 99.06 0)
 			(effects
@@
 			)
 		)
-		(property "Footprint" ""
+		(property "Footprint" "HiroFootprints:Mesa 588536"
 			(at 142.24 99.06 0)
 			(effects
@@
 			)
 		)
-		(property "Footprint" ""
+		(property "Footprint" "HiroFootprints:MB Inductor"
 			(at 163.83 121.92 0)
 			(effects
@@
 			)
 		)
-		(property "Footprint" ""
+		(property "Footprint" "HiroFootprints:MB Inductor"
 			(at 130.81 121.92 0)
 			(effects
@@
 			)
 		)
-		(property "Footprint" ""
+		(property "Footprint" "HiroFootprints:Mesa 588536"
 			(at 93.98 99.06 0)
 			(effects
@@
 			)
 		)
-		(property "Footprint" ""
+		(property "Footprint" "HiroFootprints:Mesa 588536"
 			(at 109.22 99.06 0)
 			(effects
@@
 			)
 		)
-		(property "Footprint" ""
+		(property "Footprint" "HiroFootprints:MB Inductor"
 			(at 147.32 121.92 0)
 			(effects
@@
 			)
 		)
-		(property "Footprint" ""
+		(property "Footprint" "HiroFootprints:Mesa 588536"
 			(at 125.73 99.06 0)
 			(effects

Commit message: Finished EQ Slider V1 Board
Parts:
- C4: footprint (none) -> Capacitor_THT:CP_Radial_Tantal_D4.5mm_P5.00mm
Changed lines of the file:
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@@
 			)
 		)
-		(property "Footprint" ""
+		(property "Footprint" "Capacitor_THT:CP_Radial_Tantal_D4.5mm_P5.00mm"
 			(at 146.3548 128.27 0)
 			(effects
