File: Graphic EQ/EQ_Slider_V1.0/EQ_Slider_V1.0.kicad_pcb (KiCad board)
At the start: 2 copper layers, 101.6 x 63.5 mm, 27 parts

Commit message: Added Comments to EQ Slider PCB
Other:
- board text added: "2200Hz"
- board text added: "240Hz"
- board text added: "6600Hz"
- board text added: "750Hz"
- board text added: "80Hz"
Changed lines of the file:
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@@
+		)
+	)
+	(gr_text "80Hz"
+		(at 187.68 127.26 0)
+		(layer "B.SilkS")
+		(effects
+			(font
+				(size 1.5 1.5)
+				(thickness 0.3)
+				(bold yes)
+			)
+			(justify left bottom mirror)
+		)
+	)
+	(gr_text "2200Hz"
+		(at 141.73 127.26 0)
+		(layer "B.SilkS")
+		(effects
+			(font
+				(size 1.5 1.5)
+				(thickness 0.3)
+				(bold yes)
+			)
+			(justify left bottom mirror)
+		)
+	)
+	(gr_text "240Hz"
+		(at 172.93 127.26 0)
+		(layer "B.SilkS")
+		(effects
+			(font
+				(size 1.5 1.5)
+				(thickness 0.3)
+				(bold yes)
+			)
+			(justify left bottom mirror)
+		)
+	)
+	(gr_text "6600Hz"
+		(at 126.81 127.26 0)
+		(layer "B.SilkS")
+		(effects
+			(font
+				(size 1.5 1.5)
+				(thickness 0.3)
+				(bold yes)
+			)
+			(justify left bottom mirror)
+		)
+	)
+	(gr_text "750Hz"
+		(at 157.44 127.26 0)
+		(layer "B.SilkS")
+		(effects
+			(font
+				(size 1.5 1.5)
+				(thickness 0.3)
+				(bold yes)
+			)
+			(justify left bottom mirror)
 		)
 	)
