File: Graphic EQ/EQ_Driver_V1.0/EQ_Driver_V1.0.kicad_pcb (KiCad board)
At the start: 2 copper layers, 127 x 57.2 mm, 34 parts, among them Q1 MPSA63, Q2 MPSA70, Q3 MPSA70, Q4 MPSA20

Commit message: Updated Driver V1.0 Gerber
Parts:
- added TP7: Shield, HiroFootprints:Out_Hole_3.4_1.8, F.Cu at (131.2, 75.9)
Routing:
- net GND: track 193.0 -> 198.5 mm
Changed lines of the file:
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@@
 		(property ki_fp_filters "Pin* Test*")
 		(sheetname "/")
-		(sheetfile "EQ_Driver_Board.kicad_sch")
+		(sheetfile "EQ_Driver_V1.0.kicad_sch")
 		(attr through_hole)
 		(fp_circle
@@
 		(property ki_fp_filters "Pin* Test*")
 		(sheetname "/")
-		(sheetfile "EQ_Driver_Board.kicad_sch")
+		(sheetfile "EQ_Driver_V1.0.kicad_sch")
 		(attr through_hole)
 		(fp_circle
@@
 		(property ki_fp_filters "TO?92*")
 		(sheetname "/")
-		(sheetfile "EQ_Driver_Board.kicad_sch")
+		(sheetfile "EQ_Driver_V1.0.kicad_sch")
 		(attr through_hole)
 		(fp_line
@@
 		(property ki_fp_filters "CP_*")
 		(sheetname "/")
-		(sheetfile "EQ_Driver_Board.kicad_sch")
+		(sheetfile "EQ_Driver_V1.0.kicad_sch")
 		(attr through_hole)
 		(fp_line
@@
 		(property ki_fp_filters "CP_*")
 		(sheetname "/")
-		(sheetfile "EQ_Driver_Board.kicad_sch")
+		(sheetfile "EQ_Driver_V1.0.kicad_sch")
 		(attr through_hole)
 		(fp_line
@@
 		(property ki_fp_filters "R_*")
 		(sheetname "/")
-		(sheetfile "EQ_Driver_Board.kicad_sch")
+		(sheetfile "EQ_Driver_V1.0.kicad_sch")
 		(attr through_hole)
 		(fp_line
@@
 		(property ki_fp_filters "C_*")
 		(sheetname "/")
-		(sheetfile "EQ_Driver_Board.kicad_sch")
+		(sheetfile "EQ_Driver_V1.0.kicad_sch")
 		(attr through_hole)
 		(fp_line
@@
 		(property ki_fp_filters "Pin* Test*")
 		(sheetname "/")
-		(sheetfile "EQ_Driver_Board.kicad_sch")
+		(sheetfile "EQ_Driver_V1.0.kicad_sch")
 		(attr through_hole)
 		(fp_circle
@@
 		(property ki_fp_filters "R_*")
 		(sheetname "/")
-		(sheetfile "EQ_Driver_Board.kicad_sch")
+		(sheetfile "EQ_Driver_V1.0.kicad_sch")
 		(attr through_hole)
 		(fp_line
@@
 		)
 	)
+	(footprint "HiroFootprints:Out_Hole_3.4_1.8"
+		(layer "F.Cu")
+		(at 131.21 75.86)
+		(property "Reference" "TP7"
+			(at 0 -0.5 0)
+			(unlocked yes)
+			(layer "F.SilkS")
+			(hide yes)
+			(effects
+				(font
+					(size 1 1)
+					(thickness 0.1)
+				)
+			)
+		)
+		(property "Value" "Shield"
+			(at 0.07 2.79 0)
+			(unlocked yes)
+			(layer "F.SilkS")
+			(effects
+				(font
+					(size 1 1)
+					(thickness 0.15)
+				)
+			)
+		)
+		(property "Datasheet" ""
+			(at 0 0 0)
+			(unlocked yes)
+			(layer "F.Fab")
+			(hide yes)
+			(effects
+				(font
+					(size 1 1)
+					(thickness 0.15)
+				)
+			)
+		)
+		(property "Description" "test point"
+			(at 0 0 0)
+			(unlocked yes)
+			(layer "F.Fab")
+			(hide yes)
+			(effects
+				(font
+					(size 1 1)
+					(thickness 0.15)
+				)
+			)
+		)
+		(property ki_fp_filters "Pin* Test*")
+		(sheetname "/")
+		(sheetfile "EQ_Driver_V1.0.kicad_sch")
+		(attr through_hole)
+		(fp_circle
+			(center 0 0)
+			(end 1.8 0)
+			(stroke
+				(width 0.12)
+				(type solid)
+			)
+			(fill no)
+			(layer "F.SilkS")
+		)
+		(fp_line
+			(start -1.9 -0.3)
+			(end -1.9 0.3)
+			(stroke
+				(width 0.12)
+				(type solid)
+			)
+			(layer "F.Fab")
+		)
+		(fp_line
+			(start -1.9 0.3)
+			(end 1.9 0.3)
+			(stroke
+				(width 0.12)
+				(type solid)
+			)
+			(layer "F.Fab")
+		)
+		(fp_line
+			(start 1.9 -0.3)
+			(end -1.9 -0.3)
+			(stroke
+				(width 0.12)
+				(type solid)
+			)
+			(layer "F.Fab")
+		)
+		(fp_line
+			(start 1.9 0.3)
+			(end 1.9 -0.3)
+			(stroke
+				(width 0.12)
+				(type solid)
+			)
+			(layer "F.Fab")
+		)
+		(fp_text user "${REFERENCE}"
+			(at 0.5 3.5 0)
+			(layer "F.Fab")
+			(effects
+				(font
+					(size 1 1)
+					(thickness 0.15)
+				)
+			)
+		)
+		(pad "1" thru_hole circle
+			(at 0 0)
+			(size 3.4 3.4)
+			(drill 1.8)
+			(layers "*.Cu" "*.Mask")
+			(remove_unused_layers no)
+			(net 2 "GND")
+			(pinfunction "1")
+			(pintype "passive")
+		)
+		(embedded_fonts no)
+	)
 	(footprint "Resistor_THT:R_Axial_DIN0411_L9.9mm_D3.6mm_P15.24mm_Horizontal"
 		(layer "F.Cu")
@@
 		(property ki_fp_filters "R_*")
 		(sheetname "/")
-		(sheetfile "EQ_Driver_Board.kicad_sch")
+		(sheetfile "EQ_Driver_V1.0.kicad_sch")
 		(attr through_hole)
 		(fp_line
@@
 		(property ki_fp_filters "R_*")
 		(sheetname "/")
-		(sheetfile "EQ_Driver_Board.kicad_sch")
+		(sheetfile "EQ_Driver_V1.0.kicad_sch")
 		(attr through_hole)
 		(fp_line
@@
 		(property ki_fp_filters "R_*")
 		(sheetname "/")
-		(sheetfile "EQ_Driver_Board.kicad_sch")
+		(sheetfile "EQ_Driver_V1.0.kicad_sch")
 		(attr through_hole)
 		(fp_line
@@
 		(property ki_fp_filters "C_*")
 		(sheetname "/")
-		(sheetfile "EQ_Driver_Board.kicad_sch")
+		(sheetfile "EQ_Driver_V1.0.kicad_sch")
 		(attr through_hole)
 		(fp_rect
@@
 		(property ki_fp_filters "TO?92*")
 		(sheetname "/")
-		(sheetfile "EQ_Driver_Board.kicad_sch")
+		(sheetfile "EQ_Driver_V1.0.kicad_sch")
 		(attr through_hole)
 		(fp_line
@@
 		(property ki_fp_filters "R_*")
 		(sheetname "/")
-		(sheetfile "EQ_Driver_Board.kicad_sch")
+		(sheetfile "EQ_Driver_V1.0.kicad_sch")
 		(attr through_hole)
 		(fp_line
@@
 		(property ki_fp_filters "TO?92*")
 		(sheetname "/")
-		(sheetfile "EQ_Driver_Board.kicad_sch")
+		(sheetfile "EQ_Driver_V1.0.kicad_sch")
 		(attr through_hole)
 		(fp_line
@@
 		(property ki_fp_filters "R_*")
 		(sheetname "/")
-		(sheetfile "EQ_Driver_Board.kicad_sch")
+		(sheetfile "EQ_Driver_V1.0.kicad_sch")
 		(attr through_hole)
 		(fp_line
@@
 		(property ki_fp_filters "Pin* Test*")
 		(sheetname "/")
-		(sheetfile "EQ_Driver_Board.kicad_sch")
+		(sheetfile "EQ_Driver_V1.0.kicad_sch")
 		(attr through_hole)
 		(fp_circle
@@
 		(property ki_fp_filters "TO?92*")
 		(sheetname "/")
-		(sheetfile "EQ_Driver_Board.kicad_sch")
+		(sheetfile "EQ_Driver_V1.0.kicad_sch")
 		(attr through_hole)
 		(fp_line
@@
 		(property ki_fp_filters "Pin* Test*")
 		(sheetname "/")
-		(sheetfile "EQ_Driver_Board.kicad_sch")
+		(sheetfile "EQ_Driver_V1.0.kicad_sch")
 		(attr through_hole)
 		(fp_circle
@@
 		(property ki_fp_filters "CP_*")
 		(sheetname "/")
-		(sheetfile "EQ_Driver_Board.kicad_sch")
+		(sheetfile "EQ_Driver_V1.0.kicad_sch")
 		(attr through_hole)
 		(fp_line
@@
 		(property ki_fp_filters "R_*")
 		(sheetname "/")
-		(sheetfile "EQ_Driver_Board.kicad_sch")
+		(sheetfile "EQ_Driver_V1.0.kicad_sch")
 		(attr through_hole)
 		(fp_line
@@
 		(property ki_fp_filters "R_*")
 		(sheetname "/")
-		(sheetfile "EQ_Driver_Board.kicad_sch")
+		(sheetfile "EQ_Driver_V1.0.kicad_sch")
 		(attr through_hole)
 		(fp_line
@@
 		(property ki_fp_filters "CP_*")
 		(sheetname "/")
-		(sheetfile "EQ_Driver_Board.kicad_sch")
+		(sheetfile "EQ_Driver_V1.0.kicad_sch")
 		(attr through_hole)
 		(fp_line
@@
 		(property ki_fp_filters "R_*")
 		(sheetname "/")
-		(sheetfile "EQ_Driver_Board.kicad_sch")
+		(sheetfile "EQ_Driver_V1.0.kicad_sch")
 		(attr through_hole)
 		(fp_line
@@
 		(property ki_fp_filters "R_*")
 		(sheetname "/")
-		(sheetfile "EQ_Driver_Board.kicad_sch")
+		(sheetfile "EQ_Driver_V1.0.kicad_sch")
 		(attr through_hole)
 		(fp_line
@@
 		(property ki_fp_filters "C_*")
 		(sheetname "/")
-		(sheetfile "EQ_Driver_Board.kicad_sch")
+		(sheetfile "EQ_Driver_V1.0.kicad_sch")
 		(attr through_hole)
 		(fp_line
@@
 		(property ki_fp_filters "Pin* Test*")
 		(sheetname "/")
-		(sheetfile "EQ_Driver_Board.kicad_sch")
+		(sheetfile "EQ_Driver_V1.0.kicad_sch")
 		(attr through_hole)
 		(fp_circle
@@
 	)
 	(segment
+		(start 131.21 70.44)
+		(end 131.27 70.38)
+		(width 1.6)
+		(layer "F.Cu")
+		(net 2)
+	)
+	(segment
 		(start 93.56 79.64)
 		(end 97.58 75.62)
@@
 	)
 	(segment
+		(start 131.21 75.86)
+		(end 131.21 70.44)
+		(width 1.6)
+		(layer "F.Cu")
+		(net 2)
+	)
+	(segment
 		(start 97.58 70.38)
 		(end 103.12 70.38)
@@
 	)
 	(segment
+		(start 131.27 70.38)
+		(end 151.08 70.38)
+		(width 1.6)
+		(layer "F.Cu")
+		(net 2)
+	)
+	(segment
 		(start 126.31 70.44)
 		(end 126.37 70.38)
@@
 	(segment
 		(start 126.37 70.38)
-		(end 151.08 70.38)
+		(end 131.27 70.38)
 		(width 1.6)
 		(layer "F.Cu")
