File: Graphic EQ/EQ_Driver_V1.0/EQ_Driver_V1.0.kicad_sch (KiCad schematic)
At the start: 28 parts, among them Q1 MPSA63, Q2 MPSA70, Q3 MPSA70, Q4 MPSA20

Commit message: Updated Driver V1.0 Gerber
Parts:
- added TP7: Shield, HiroFootprints:Out_Hole_3.4_1.8, symbol Connector:TestPoint
Connections:
- net GND: now also TP7.1
Changed lines of the file:
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@@
+	)
+	(junction
+		(at 135.89 104.14)
+		(diameter 0)
+		(color 0 0 0 0)
 	)
 	(junction
@@
 	(wire
 		(pts
+			(xy 135.89 104.14) (xy 158.75 104.14)
+		)
+		(stroke
+			(width 0)
+			(type default)
+		)
+	)
+	(wire
+		(pts
 			(xy 170.18 104.14) (xy 170.18 100.33)
 		)
@@
 	(wire
 		(pts
-			(xy 130.81 104.14) (xy 158.75 104.14)
+			(xy 130.81 104.14) (xy 135.89 104.14)
 		)
 		(stroke
@@
 					(unit 1)
 				)
+			)
+		)
+	)
+	(symbol
+		(lib_id "Connector:TestPoint")
+		(at 135.89 104.14 180)
+		(unit 1)
+		(exclude_from_sim no)
+		(in_bom yes)
+		(on_board yes)
+		(dnp no)
+		(fields_autoplaced yes)
+		(property "Reference" "TP7"
+			(at 138.43 106.1719 0)
+			(effects
+				(font
+					(size 1.27 1.27)
+				)
+				(justify right)
+			)
+		)
+		(property "Value" "Shield"
+			(at 138.43 108.7119 0)
+			(effects
+				(font
+					(size 1.27 1.27)
+				)
+				(justify right)
+			)
+		)
+		(property "Footprint" "HiroFootprints:Out_Hole_3.4_1.8"
+			(at 130.81 104.14 0)
+			(effects
+				(font
+					(size 1.27 1.27)
+				)
+				(hide yes)
+			)
+		)
+		(property "Datasheet" "~"
+			(at 130.81 104.14 0)
+			(effects
+				(font
+					(size 1.27 1.27)
+				)
+				(hide yes)
+			)
+		)
+		(property "Description" "test point"
+			(at 135.89 104.14 0)
+			(effects
+				(font
+					(size 1.27 1.27)
+				)
+				(hide yes)
+			)
+		)
+		(pin "1"
+		)
+		(instances
+			(project "EQ_Driver_V1.0"
+				(path "/8b3e6737-4f8d-464d-ab54-70eaaf54bfcf"
+					(reference "TP7")
+					(unit 1)
+				)

Commit message: Started Power Supply Board, Made EQ Driver Changes
Parts:
- R11: footprint Resistor_THT:R_Axial_DIN0411_L9.9mm_D3.6mm_P15.24mm_Horizontal -> Resistor_THT:R_Axial_DIN0516_L15.5mm_D5.0mm_P20.32mm_Horizontal
Changed lines of the file:
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@@
 			)
 		)
-		(property "Footprint" "Resistor_THT:R_Axial_DIN0411_L9.9mm_D3.6mm_P15.24mm_Horizontal"
+		(property "Footprint" "Resistor_THT:R_Axial_DIN0516_L15.5mm_D5.0mm_P20.32mm_Horizontal"
 			(at 182.88 60.198 90)
 			(effects

Commit message: Added Solder Pads, Updated Power Supply Board
Parts:
- TP1, TP2, TP3, TP6, TP7: footprint HiroFootprints:Out_Hole_3.4_1.8 -> HiroFootprints:WirePad
Changed lines of the file:
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@@
 			)
 		)
-		(property "Footprint" "HiroFootprints:Out_Hole_3.4_1.8"
+		(property "Footprint" "HiroFootprints:WirePad"
 			(at 143.51 111.76 0)
 			(effects
@@
 			)
 		)
-		(property "Footprint" "HiroFootprints:Out_Hole_3.4_1.8"
+		(property "Footprint" "HiroFootprints:WirePad"
 			(at 66.04 77.47 0)
 			(effects
@@
 			)
 		)
-		(property "Footprint" "HiroFootprints:Out_Hole_3.4_1.8"
+		(property "Footprint" "HiroFootprints:WirePad"
 			(at 109.22 111.76 0)
 			(effects
@@
 			)
 		)
-		(property "Footprint" "HiroFootprints:Out_Hole_3.4_1.8"
+		(property "Footprint" "HiroFootprints:WirePad"
 			(at 130.81 104.14 0)
 			(effects
@@
 			)
 		)
-		(property "Footprint" "HiroFootprints:Out_Hole_3.4_1.8"
+		(property "Footprint" "HiroFootprints:WirePad"
 			(at 180.34 72.39 0)
 			(effects

Commit message: Updated Ceramic Capacitor Footprints
Parts:
- C3, C4: footprint Capacitor_THT:C_Rect_L11.0mm_W3.5mm_P10.00mm_MKT -> HiroFootprints:10_47_120_180_250_500pF_1KV_Cer_6.4_4.0_6.4
Changed lines of the file:
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@@
 			)
 		)
-		(property "Footprint" "Capacitor_THT:C_Rect_L11.0mm_W3.5mm_P10.00mm_MKT"
+		(property "Footprint" "HiroFootprints:10_47_120_180_250_500pF_1KV_Cer_6.4_4.0_6.4"
 			(at 157.48 91.1352 0)
 			(effects
@@
 			)
 		)
-		(property "Footprint" "Capacitor_THT:C_Rect_L11.0mm_W3.5mm_P10.00mm_MKT"
+		(property "Footprint" "HiroFootprints:10_47_120_180_250_500pF_1KV_Cer_6.4_4.0_6.4"
 			(at 152.4 71.4248 0)
 			(effects

Commit message: Adjusted Resistor Sizes
Parts:
- R1, R10, R2, R3: footprint Resistor_THT:R_Axial_DIN0411_L9.9mm_D3.6mm_P15.24mm_Horizontal -> Resistor_THT:R_Axial_DIN0309_L9.0mm_D3.2mm_P12.70mm_Horizontal
- R4, R5, R6, R7, R8, R9: footprint Resistor_THT:R_Axial_DIN0411_L9.9mm_D3.6mm_P15.24mm_Horizontal -> Resistor_THT:R_Axial_DIN0414_L11.9mm_D4.5mm_P15.24mm_Horizontal
Changed lines of the file:
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@@
 			)
 		)
-		(property "Footprint" "Resistor_THT:R_Axial_DIN0411_L9.9mm_D3.6mm_P15.24mm_Horizontal"
+		(property "Footprint" "Resistor_THT:R_Axial_DIN0414_L11.9mm_D4.5mm_P15.24mm_Horizontal"
 			(at 129.032 96.52 90)
 			(effects
@@
 			)
 		)
-		(property "Footprint" "Resistor_THT:R_Axial_DIN0411_L9.9mm_D3.6mm_P15.24mm_Horizontal"
+		(property "Footprint" "Resistor_THT:R_Axial_DIN0414_L11.9mm_D4.5mm_P15.24mm_Horizontal"
 			(at 156.972 96.52 90)
 			(effects
@@
 			)
 		)
-		(property "Footprint" "Resistor_THT:R_Axial_DIN0411_L9.9mm_D3.6mm_P15.24mm_Horizontal"
+		(property "Footprint" "Resistor_THT:R_Axial_DIN0414_L11.9mm_D4.5mm_P15.24mm_Horizontal"
 			(at 153.67 84.328 90)
 			(effects
@@
 			)
 		)
-		(property "Footprint" "Resistor_THT:R_Axial_DIN0411_L9.9mm_D3.6mm_P15.24mm_Horizontal"
+		(property "Footprint" "Resistor_THT:R_Axial_DIN0414_L11.9mm_D4.5mm_P15.24mm_Horizontal"
 			(at 109.22 85.852 90)
 			(effects
@@
 			)
 		)
-		(property "Footprint" "Resistor_THT:R_Axial_DIN0411_L9.9mm_D3.6mm_P15.24mm_Horizontal"
+		(property "Footprint" "Resistor_THT:R_Axial_DIN0309_L9.0mm_D3.2mm_P12.70mm_Horizontal"
 			(at 85.852 96.52 90)
 			(effects
@@
 			)
 		)
-		(property "Footprint" "Resistor_THT:R_Axial_DIN0411_L9.9mm_D3.6mm_P15.24mm_Horizontal"
+		(property "Footprint" "Resistor_THT:R_Axial_DIN0414_L11.9mm_D4.5mm_P15.24mm_Horizontal"
 			(at 95.25 60.198 90)
 			(effects
@@
 			)
 		)
-		(property "Footprint" "Resistor_THT:R_Axial_DIN0411_L9.9mm_D3.6mm_P15.24mm_Horizontal"
+		(property "Footprint" "Resistor_THT:R_Axial_DIN0309_L9.0mm_D3.2mm_P12.70mm_Horizontal"
 			(at 71.882 96.52 90)
 			(effects
@@
 			)
 		)
-		(property "Footprint" "Resistor_THT:R_Axial_DIN0411_L9.9mm_D3.6mm_P15.24mm_Horizontal"
+		(property "Footprint" "Resistor_THT:R_Axial_DIN0309_L9.0mm_D3.2mm_P12.70mm_Horizontal"
 			(at 168.402 96.52 90)
 			(effects
@@
 			)
 		)
-		(property "Footprint" "Resistor_THT:R_Axial_DIN0411_L9.9mm_D3.6mm_P15.24mm_Horizontal"
+		(property "Footprint" "Resistor_THT:R_Axial_DIN0414_L11.9mm_D4.5mm_P15.24mm_Horizontal"
 			(at 99.822 96.52 90)
 			(effects
@@
 			)
 		)
-		(property "Footprint" "Resistor_THT:R_Axial_DIN0411_L9.9mm_D3.6mm_P15.24mm_Horizontal"
+		(property "Footprint" "Resistor_THT:R_Axial_DIN0309_L9.0mm_D3.2mm_P12.70mm_Horizontal"
 			(at 85.852 69.85 90)
 			(effects
