File: Experiments/Bias_Supply_Variations/Bias_Supply_Variations.kicad_pcb (KiCad board)
At the start: 2 copper layers, 60 parts

Commit message: Created Different Bias Schematics and Layout for Future Reference
Parts:
- moved D9 236.7 mm to (28.5, 162.7)
- moved D3 235.3 mm to (20.9, 52.1)
- moved D1 234.7 mm to (20.9, 58.1)
- moved D10 234.1 mm to (28.5, 157.3)
- moved D5 230.5 mm to (28.1, 116.7)
- moved TP14 229.9 mm to (23.3, 160.1)
- moved TP3 229.2 mm to (16.6, 58.0)
- moved D7 228.7 mm to (28.1, 112.2)
- moved TP9 220.2 mm to (22.8, 113.0)
- moved R5 197.3 mm to (35.5, 52.0)
- moved R3 195.9 mm to (35.5, 58.0)
- moved R22 194.9 mm to (42.5, 163.4)
- moved R23 192.0 mm to (42.5, 156.9)
- moved R13 191.4 mm to (42.3, 118.7)
- moved R15 189.3 mm to (42.3, 112.0)
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Routing:
- net G: track 0.00 -> 172.4 mm
- net F: track 0.00 -> 129.9 mm
- net 60VAC: track 0.00 -> 55.7 mm
- net Net-(C2-Pad2): track 0.00 -> 38.1 mm
- net Net-(C3-Pad2): track 0.00 -> 22.1 mm
- net Net-(C4-Pad2): track 0.00 -> 20.3 mm
- net Net-(C5-Pad2): track 0.00 -> 14.9 mm
- net Net-(C9-Pad2): track 0.00 -> 14.8 mm
- net Net-(C6-Pad2): track 0.00 -> 5.88 mm
- net Net-(D5-A): track 0.00 -> 4.79 mm
- net Net-(D3-A): track 0.00 -> 4.56 mm
- net Net-(D1-A): track 0.00 -> 4.54 mm
- net Net-(D6-A): track 0.00 -> 4.53 mm
- net Net-(D2-A): track 0.00 -> 4.33 mm
- net Net-(D8-A): track 0.00 -> 4.30 mm
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Other:
- board text added: "SLOCLONE and Mesa Boogie are the SAME"
