File: Power Supply/Power_Supply_V1.0/Power_Supply_V1.0.kicad_sch (KiCad schematic)
At the start: 38 parts, among them SW1 Standby

Commit message: Added Solder Pads, Updated Power Supply Board
Parts:
- added TP13: GND 3, HiroFootprints:WirePad, symbol Connector:TestPoint
- added TP14: GND 4, HiroFootprints:WirePad, symbol Connector:TestPoint
- added TP15: Bias Tap Out, HiroFootprints:WirePad, symbol Connector:TestPoint
- TP12, TP3, TP4, TP5, TP6, TP7, TP8: footprint HiroFootprints:Out_Hole_3.4_1.8 -> HiroFootprints:WirePad
Connections:
- net 60VAC: now also TP15.1
- net GND: now also TP13.1, TP14.1

Commit message: Adjusted Resistor Sizes
Parts:
- R6, R7, R8: footprint Resistor_THT:R_Axial_DIN0411_L9.9mm_D3.6mm_P15.24mm_Horizontal -> Resistor_THT:R_Axial_DIN0309_L9.0mm_D3.2mm_P12.70mm_Horizontal
Changed lines of the file:
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@@
 			)
 		)
-		(property "Footprint" "Resistor_THT:R_Axial_DIN0411_L9.9mm_D3.6mm_P15.24mm_Horizontal"
+		(property "Footprint" "Resistor_THT:R_Axial_DIN0309_L9.0mm_D3.2mm_P12.70mm_Horizontal"
 			(at 132.08 176.022 90)
 			(effects
@@
 			)
 		)
-		(property "Footprint" "Resistor_THT:R_Axial_DIN0411_L9.9mm_D3.6mm_P15.24mm_Horizontal"
+		(property "Footprint" "Resistor_THT:R_Axial_DIN0309_L9.0mm_D3.2mm_P12.70mm_Horizontal"
 			(at 124.968 146.05 90)
 			(effects
@@
 			)
 		)
-		(property "Footprint" "Resistor_THT:R_Axial_DIN0411_L9.9mm_D3.6mm_P15.24mm_Horizontal"
+		(property "Footprint" "Resistor_THT:R_Axial_DIN0309_L9.0mm_D3.2mm_P12.70mm_Horizontal"
 			(at 132.08 163.322 90)
 			(effects
