File: Preamp/Preamp_Reverb_V1.0/Preamp_Reverb_V1.0.kicad_sch (KiCad schematic)
At the start: 150 parts, among them J1 Send, J2 Return, J3 Return, J4 Send, J5 Send, SW1 Pull Pot, SW2 Pull Pot, SW3 Pull Pot, SW4 Pull Pot, SW5 Pull Pot, SW6 Pull Pot, SW7 SW_SP3T, SW8 Pull Pot, SW9 Pull Pot, T1 Mesa 550185

Commit message: Updated Ceramic Capacitor Footprints
Parts:
- C1, C7: footprint (none) -> HiroFootprints:20_750pF_1KV_Cer_7.4_4.0_.6.4
- C11, C2, C21, C4, C5: footprint (none) -> HiroFootprints:715P47354LAD3
- C13, C14, C16, C25: footprint (none) -> Capacitor_THT:CP_Axial_L11.0mm_D5.0mm_P18.00mm_Horizontal
- C17, C23, C30, C6: footprint (none) -> HiroFootprints:10_47_120_180_250_500pF_1KV_Cer_6.4_4.0_6.4
- C19, C29: footprint (none) -> HiroFootprints:1000pF_1KV_Cer_9.4_4.0_6.4
- C20, C3: footprint (none) -> HiroFootprints:715P22354KAD3
- C22: footprint (none) -> HiroFootprints:715P10354JAD3
- C27, C28: footprint (none) -> Capacitor_THT:CP_Axial_L10.0mm_D4.5mm_P15.00mm_Horizontal
- C32: footprint (none) -> Capacitor_THT:CP_Axial_L18.0mm_D8.0mm_P25.00mm_Horizontal
- C9: footprint (none) -> HiroFootprints:715P10454LAD3
- D1, D6: footprint (none) -> Diode_THT:D_DO-41_SOD81_P10.16mm_Horizontal
- D5: footprint (none) -> Diode_THT:D_DO-201AE_P12.70mm_Horizontal
Changed lines of the file:
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@@
 			)
 		)
-		(property "Footprint" ""
+		(property "Footprint" "Capacitor_THT:CP_Axial_L11.0mm_D5.0mm_P18.00mm_Horizontal"
 			(at 393.3952 212.09 0)
 			(effects
@@
 			)
 		)
-		(property "Footprint" ""
+		(property "Footprint" "Diode_THT:D_DO-201AE_P12.70mm_Horizontal"
 			(at 132.08 325.12 0)
 			(effects
@@
 			)
 		)
-		(property "Footprint" ""
+		(property "Footprint" "Capacitor_THT:CP_Axial_L18.0mm_D8.0mm_P25.00mm_Horizontal"
 			(at 117.8052 328.93 0)
 			(effects
@@
 			)
 		)
-		(property "Footprint" ""
+		(property "Footprint" "HiroFootprints:715P47354LAD3"
 			(at 388.62 65.0748 0)
 			(effects
@@
 			)
 		)
-		(property "Footprint" ""
+		(property "Footprint" "HiroFootprints:10_47_120_180_250_500pF_1KV_Cer_6.4_4.0_6.4"
 			(at 161.29 76.5048 0)
 			(effects
@@
 			)
 		)
-		(property "Footprint" ""
+		(property "Footprint" "HiroFootprints:715P10354JAD3"
 			(at 393.7 179.3748 0)
 			(effects
@@
 			)
 		)
-		(property "Footprint" ""
+		(property "Footprint" "HiroFootprints:10_47_120_180_250_500pF_1KV_Cer_6.4_4.0_6.4"
 			(at 279.0952 121.92 0)
 			(effects
@@
 			)
 		)
-		(property "Footprint" ""
+		(property "Footprint" "HiroFootprints:715P10454LAD3"
 			(at 161.29 87.9348 0)
 			(effects
@@
 			)
 		)
-		(property "Footprint" ""
+		(property "Footprint" "HiroFootprints:1000pF_1KV_Cer_9.4_4.0_6.4"
 			(at 183.8452 224.79 0)
 			(effects
@@
 			)
 		)
-		(property "Footprint" ""
+		(property "Footprint" "HiroFootprints:715P47354LAD3"
 			(at 227.33 178.1048 0)
 			(effects
@@
 			)
 		)
-		(property "Footprint" ""
+		(property "Footprint" "HiroFootprints:1000pF_1KV_Cer_9.4_4.0_6.4"
 			(at 200.3552 173.99 0)
 			(effects
@@
 			)
 		)
-		(property "Footprint" ""
+		(property "Footprint" "HiroFootprints:20_750pF_1KV_Cer_7.4_4.0_.6.4"
 			(at 250.19 81.5848 0)
 			(effects
@@
 			)
 		)
-		(property "Footprint" ""
+		(property "Footprint" "HiroFootprints:10_47_120_180_250_500pF_1KV_Cer_6.4_4.0_6.4"
 			(at 245.11 189.5348 0)
 			(effects
@@
 			)
 		)
-		(property "Footprint" ""
+		(property "Footprint" "Capacitor_THT:CP_Axial_L10.0mm_D4.5mm_P15.00mm_Horizontal"
 			(at 157.1752 224.79 0)
 			(effects
@@
 			)
 		)
-		(property "Footprint" ""
+		(property "Footprint" "HiroFootprints:715P47354LAD3"
 			(at 161.29 99.3648 0)
 			(effects
@@
 			)
 		)
-		(property "Footprint" ""
+		(property "Footprint" "HiroFootprints:715P22354KAD3"
 			(at 171.45 178.1048 0)
 			(effects
@@
 			)
 		)
-		(property "Footprint" ""
+		(property "Footprint" "HiroFootprints:715P47354LAD3"
 			(at 223.52 67.0052 0)
 			(effects
@@
 			)
 		)
-		(property "Footprint" ""
+		(property "Footprint" "Capacitor_THT:CP_Axial_L10.0mm_D4.5mm_P15.00mm_Horizontal"
 			(at 333.7052 223.52 0)
 			(effects
@@
 			)
 		)
-		(property "Footprint" ""
+		(property "Footprint" "HiroFootprints:715P47354LAD3"
 			(at 295.91 65.0748 0)
 			(effects
@@
 			)
 		)
-		(property "Footprint" ""
+		(property "Footprint" "HiroFootprints:715P22354KAD3"
 			(at 236.22 65.0748 0)
 			(effects
@@
 			)
 		)
-		(property "Footprint" ""
+		(property "Footprint" "HiroFootprints:10_47_120_180_250_500pF_1KV_Cer_6.4_4.0_6.4"
 			(at 238.4552 224.79 0)
 			(effects
@@
 			)
 		)
-		(property "Footprint" ""
+		(property "Footprint" "Diode_THT:D_DO-41_SOD81_P10.16mm_Horizontal"
 			(at 207.01 349.25 0)
 			(effects
@@
 			)
 		)
-		(property "Footprint" ""
+		(property "Footprint" "HiroFootprints:20_750pF_1KV_Cer_7.4_4.0_.6.4"
 			(at 161.29 65.0748 0)
 			(effects
@@
 			)
 		)
-		(property "Footprint" ""
+		(property "Footprint" "Capacitor_THT:CP_Axial_L11.0mm_D5.0mm_P18.00mm_Horizontal"
 			(at 374.3452 107.95 0)
 			(effects
@@
 			)
 		)
-		(property "Footprint" ""
+		(property "Footprint" "Capacitor_THT:CP_Axial_L11.0mm_D5.0mm_P18.00mm_Horizontal"
 			(at 205.4352 121.92 0)
 			(effects
@@
 			)
 		)
-		(property "Footprint" ""
+		(property "Footprint" "Diode_THT:D_DO-41_SOD81_P10.16mm_Horizontal"
 			(at 173.99 260.35 0)
 			(effects
@@
 			)
 		)
-		(property "Footprint" ""
+		(property "Footprint" "Capacitor_THT:CP_Axial_L11.0mm_D5.0mm_P18.00mm_Horizontal"
 			(at 122.8852 109.22 0)
 			(effects

Commit message: Adjusted Resistor Sizes
Parts:
- C15, C18: footprint (none) -> Capacitor_THT:C_Rect_L7.2mm_W4.5mm_P5.00mm_FKS2_FKP2_MKS2_MKP2
Changed lines of the file:
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@@
 			)
 		)
-		(property "Footprint" ""
+		(property "Footprint" "Capacitor_THT:C_Rect_L7.2mm_W4.5mm_P5.00mm_FKS2_FKP2_MKS2_MKP2"
 			(at 398.4752 121.92 0)
 			(effects
@@
 			)
 		)
-		(property "Footprint" ""
+		(property "Footprint" "Capacitor_THT:C_Rect_L7.2mm_W4.5mm_P5.00mm_FKS2_FKP2_MKS2_MKP2"
 			(at 147.0152 121.92 0)
 			(effects

Commit message: Preamp Progress, and Custom Footprint Library
Parts:
- C10: footprint (none) -> Capacitor_THT:CP_Axial_L11.0mm_D5.0mm_P18.00mm_Horizontal
- C12: footprint (none) -> HiroFootprints:20_750pF_1KV_Cer_7.4_4.0_.6.4
- C24: footprint (none) -> Capacitor_THT:CP_Axial_L10.0mm_D4.5mm_P15.00mm_Horizontal
- D5: footprint Diode_THT:D_DO-201AE_P12.70mm_Horizontal -> Diode_THT:D_DO-201_P15.24mm_Horizontal
- J3: value Return -> Reverb FS
- J4: value Send -> EQ FS
- J5: value Send -> Lead FS
- R1, R2, R24, R3: footprint Resistor_THT:R_Axial_DIN0411_L9.9mm_D3.6mm_P15.24mm_Horizontal -> Resistor_THT:R_Axial_DIN0516_L15.5mm_D5.0mm_P20.32mm_Horizontal
- R10, R18, R22, R29, R32, R35, R39, R41, R45, R46, R49, R5, R51, R6: footprint Resistor_THT:R_Axial_DIN0411_L9.9mm_D3.6mm_P15.24mm_Horizontal -> Resistor_THT:R_Axial_DIN0414_L11.9mm_D4.5mm_P15.24mm_Horizontal
- R11, R14, R15, R16, R17, R20, R25, R26, R27, R30, R31, R33, R34, R37, R38, R4, R42, R9: footprint Resistor_THT:R_Axial_DIN0411_L9.9mm_D3.6mm_P15.24mm_Horizontal -> Resistor_THT:R_Axial_DIN0309_L9.0mm_D3.2mm_P12.70mm_Horizontal
- R12: footprint (none) -> Resistor_THT:R_Axial_DIN0414_L11.9mm_D4.5mm_P15.24mm_Horizontal
- R43, R44, R50: footprint Resistor_THT:R_Axial_DIN0411_L9.9mm_D3.6mm_P15.24mm_Horizontal -> (none)
- R7: footprint Resistor_THT:R_Axial_DIN0411_L9.9mm_D3.6mm_P15.24mm_Horizontal -> Resistor_THT:R_Axial_DIN0617_L17.0mm_D6.0mm_P25.40mm_Horizontal
- TP1, TP10, TP11, TP12, TP13, TP14, TP15, TP16, TP17, TP18, TP19, TP2, TP20, TP21, TP22, TP23, TP24, TP25, TP26, TP27, TP29, TP3, TP4, TP5, TP6, TP7, TP8, TP9: footprint HiroFootprints:Out_Hole_3.4_1.8 -> (none)
- TP28: value L FS -> Lead FS; footprint HiroFootprints:Out_Hole_3.4_1.8 -> (none)
- V1, V2, V3, V4: footprint Valve:Valve_Noval_P -> Valve:Valve_ECC-83-2
Connections:
- net Input: now also V1.2 (G); no longer V1.7 (G)
- net Lead Out: now also V2.7 (G); no longer V2.2 (G)
- net Tank Out: now also V3.2 (G); no longer V3.7 (G)
- net at C25.1, R35.1: now also V3.3 (K); no longer V3.8 (K)
- net at C2.2, C3.1, C7.1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: no longer TP7.1
- net at C22.1, R24.2: now also V3.1 (A); no longer V3.6 (A)
- net at C29.1, R29.2, R39.1: now also V4.2 (G); no longer V4.7 (G)
- net at C19.2, C21.1, R26.2: now also V4.1 (A); no longer V4.6 (A)
- net at C5.1, R4.2: now also V2.1 (A); no longer V2.6 (A)
- net at C1.1, C6.1, R1.2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: now also V1.1 (A); no longer V1.6 (A)
- net at C26.1, R37.1, RV8.2: now also V3.7 (G); no longer V3.2 (G)
- net at J2.T, R22.1: now also V2.2 (G); no longer V2.7 (G)
- net at C13.1, C18.1, R20.1: now also V2.3 (K); no longer V2.8 (K)
- net at C12.2, SW2.1 (A): now also TP7.1
- net at C4.1, R3.2: now also V2.6 (A); no longer V2.1 (A)
- net at C10.1, R11.1: now also V2.8 (K); no longer TP11.1, V2.3 (K)
- net at C16.1, R16.1: now also V1.8 (K); no longer V1.3 (K)
- net at C26.2, C28.1, R38.1: now also V3.8 (K); no longer V3.3 (K)
- net at C20.1, R25.2: now also V3.6 (A); no longer V3.1 (A)
- net at R30.2, R31.1: now also V4.7 (G); no longer V4.2 (G)
- net at C2.1, R2.2: now also V1.6 (A); no longer V1.1 (A)
- net at RV5.2, SW1.1 (A): now also V1.7 (G); no longer V1.2 (G)
- net at C10.2, SW3.1 (A): now also TP11.1
- net at C27.1, R32.1: now also V4.8 (K); no longer V4.3 (K)
- net at C14.1, C15.1, R15.1: now also V1.3 (K); no longer V1.8 (K)
- net at C24.1, R41.1: now also V4.3 (K); no longer V4.8 (K)
- net at T1.2 (AB): now also V4.6 (A); no longer V4.1 (A)
Other:
- note added: "X?"
- moved on the sheet: TP11, TP7, V1A, V1B, V2A, V2B, V3A, V3B, V4A, V4B

Commit message: Updated 12AX7 footprint, resized preamp board
Parts:
- V1, V2, V3, V4: footprint Valve:Valve_ECC-83-2 -> IICPP_Clone_Footprints:VT9-ST-C
Changed lines of the file:
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@@
 			)
 		)
-		(property "Footprint" "Valve:Valve_ECC-83-2"
+		(property "Footprint" "IICPP_Clone_Footprints:VT9-ST-C"
 			(at 377.698 316.23 0)
 			(effects
@@
 			)
 		)
-		(property "Footprint" "Valve:Valve_ECC-83-2"
+		(property "Footprint" "IICPP_Clone_Footprints:VT9-ST-C"
 			(at 161.798 201.93 0)
 			(effects
@@
 			)
 		)
-		(property "Footprint" "Valve:Valve_ECC-83-2"
+		(property "Footprint" "IICPP_Clone_Footprints:VT9-ST-C"
 			(at 286.258 91.44 0)
 			(effects
@@
 			)
 		)
-		(property "Footprint" "Valve:Valve_ECC-83-2"
+		(property "Footprint" "IICPP_Clone_Footprints:VT9-ST-C"
 			(at 378.968 91.44 0)
 			(effects
@@
 			)
 		)
-		(property "Footprint" "Valve:Valve_ECC-83-2"
+		(property "Footprint" "IICPP_Clone_Footprints:VT9-ST-C"
 			(at 356.108 316.23 0)
 			(effects
@@
 			)
 		)
-		(property "Footprint" "Valve:Valve_ECC-83-2"
+		(property "Footprint" "IICPP_Clone_Footprints:VT9-ST-C"
 			(at 399.288 316.23 0)
 			(effects
@@
 			)
 		)
-		(property "Footprint" "Valve:Valve_ECC-83-2"
+		(property "Footprint" "IICPP_Clone_Footprints:VT9-ST-C"
 			(at 137.668 91.44 0)
 			(effects
@@
 			)
 		)
-		(property "Footprint" "Valve:Valve_ECC-83-2"
+		(property "Footprint" "IICPP_Clone_Footprints:VT9-ST-C"
 			(at 218.948 91.44 0)
 			(effects
@@
 			)
 		)
-		(property "Footprint" "Valve:Valve_ECC-83-2"
+		(property "Footprint" "IICPP_Clone_Footprints:VT9-ST-C"
 			(at 218.948 201.93 0)
 			(effects
@@
 			)
 		)
-		(property "Footprint" "Valve:Valve_ECC-83-2"
+		(property "Footprint" "IICPP_Clone_Footprints:VT9-ST-C"
 			(at 420.878 316.23 0)
 			(effects
@@
 			)
 		)
-		(property "Footprint" "Valve:Valve_ECC-83-2"
+		(property "Footprint" "IICPP_Clone_Footprints:VT9-ST-C"
 			(at 347.218 200.66 0)
 			(effects
@@
 			)
 		)
-		(property "Footprint" "Valve:Valve_ECC-83-2"
+		(property "Footprint" "IICPP_Clone_Footprints:VT9-ST-C"
 			(at 387.858 200.66 0)
 			(effects
