File: Preamp/Preamp_Reverb_V1.0/Preamp_Reverb_V1.0.kicad_pcb (KiCad board)
At the start: 2 copper layers, 110 parts

Commit message: Preamp Progress, and Custom Footprint Library
Parts:
- removed R43: 680, Resistor_THT:R_Axial_DIN0411_L9.9mm_D3.6mm_P15.24mm_Horizontal
- removed R44: 220, Resistor_THT:R_Axial_DIN0411_L9.9mm_D3.6mm_P15.24mm_Horizontal
- removed R50: 100, Resistor_THT:R_Axial_DIN0411_L9.9mm_D3.6mm_P15.24mm_Horizontal
- removed TP1: GND, HiroFootprints:Out_Hole_3.4_1.8
- removed TP10: PBright, HiroFootprints:Out_Hole_3.4_1.8
- removed TP11: CPP2 Out, HiroFootprints:Out_Hole_3.4_1.8
- removed TP12: CPP2 In, HiroFootprints:Out_Hole_3.4_1.8
- removed TP13: LM Out, HiroFootprints:Out_Hole_3.4_1.8
- removed TP14: LM In, HiroFootprints:Out_Hole_3.4_1.8
- removed TP15: RVPot, HiroFootprints:Out_Hole_3.4_1.8
- removed TP16: PDeep, HiroFootprints:Out_Hole_3.4_1.8
- removed TP17: To GEQ, HiroFootprints:Out_Hole_3.4_1.8
- removed TP18: Mas1, HiroFootprints:Out_Hole_3.4_1.8
- removed TP19: 60VAC, HiroFootprints:Out_Hole_3.4_1.8
- removed TP2: D, HiroFootprints:Out_Hole_3.4_1.8
- removed TP20: EQ In, HiroFootprints:Out_Hole_3.4_1.8
- removed TP21: EQ Auto, HiroFootprints:Out_Hole_3.4_1.8
- removed TP22: EQ FS, HiroFootprints:Out_Hole_3.4_1.8
- removed TP23: EQ SW, HiroFootprints:Out_Hole_3.4_1.8
- removed TP24: GEQ, HiroFootprints:Out_Hole_3.4_1.8
- removed TP25: RV FS, HiroFootprints:Out_Hole_3.4_1.8
- removed TP26: TShift 1, HiroFootprints:Out_Hole_3.4_1.8
- removed TP27: TShift 2, HiroFootprints:Out_Hole_3.4_1.8
- removed TP28: L FS, HiroFootprints:Out_Hole_3.4_1.8
- removed TP29: PLead, HiroFootprints:Out_Hole_3.4_1.8
- removed TP3: BShift, HiroFootprints:Out_Hole_3.4_1.8
- removed TP4: TPot, HiroFootprints:Out_Hole_3.4_1.8
- removed TP5: BPot, HiroFootprints:Out_Hole_3.4_1.8
- removed TP6: MPot, HiroFootprints:Out_Hole_3.4_1.8
- removed TP7: CPP1 Out, HiroFootprints:Out_Hole_3.4_1.8
- removed TP8: CPP1 In, HiroFootprints:Out_Hole_3.4_1.8
- removed TP9: 680K/1M, HiroFootprints:Out_Hole_3.4_1.8
- added C10: 15uF, Capacitor_THT:CP_Axial_L11.0mm_D5.0mm_P18.00mm_Horizontal, F.Cu at (204.0, 64.3)
- added C12: 10/20pF, HiroFootprints:20_750pF_1KV_Cer_7.4_4.0_.6.4, F.Cu at (209.0, 71.8)
- added C15: 0.47uF, Capacitor_THT:C_Rect_L7.2mm_W4.5mm_P5.00mm_FKS2_FKP2_MKS2_MKP2, F.Cu at (300.8, 124.3)
- added C18: 0.47uF, Capacitor_THT:C_Rect_L7.2mm_W4.5mm_P5.00mm_FKS2_FKP2_MKS2_MKP2, F.Cu at (247.8, 130.6)
- added C24: 220nF, Capacitor_THT:CP_Axial_L10.0mm_D4.5mm_P15.00mm_Horizontal, F.Cu at (134.0, 144.7)
- added R12: 3M3, Resistor_THT:R_Axial_DIN0414_L11.9mm_D4.5mm_P15.24mm_Horizontal, F.Cu at (204.2, 78.6)
- D5: footprint Diode_THT:D_DO-201AE_P12.70mm_Horizontal -> Diode_THT:D_DO-201_P15.24mm_Horizontal
- R1, R2, R24, R3: footprint Resistor_THT:R_Axial_DIN0411_L9.9mm_D3.6mm_P15.24mm_Horizontal -> Resistor_THT:R_Axial_DIN0516_L15.5mm_D5.0mm_P20.32mm_Horizontal
- R10, R18, R22, R29, R32, R35, R39, R41, R45, R46, R49, R5, R51, R6: footprint Resistor_THT:R_Axial_DIN0411_L9.9mm_D3.6mm_P15.24mm_Horizontal -> Resistor_THT:R_Axial_DIN0414_L11.9mm_D4.5mm_P15.24mm_Horizontal
- R11, R14, R15, R16, R17, R20, R25, R26, R27, R30, R31, R33, R34, R37, R38, R4, R42, R9: footprint Resistor_THT:R_Axial_DIN0411_L9.9mm_D3.6mm_P15.24mm_Horizontal -> Resistor_THT:R_Axial_DIN0309_L9.0mm_D3.2mm_P12.70mm_Horizontal
- R7: footprint Resistor_THT:R_Axial_DIN0411_L9.9mm_D3.6mm_P15.24mm_Horizontal -> Resistor_THT:R_Axial_DIN0617_L17.0mm_D6.0mm_P25.40mm_Horizontal
- V1, V2, V3, V4: footprint Valve:Valve_Noval_P -> Valve:Valve_ECC-83-2; moved to B.Cu
- moved R7 326.9 mm to (370.6, 153.2), turned to 90 degrees
- moved R9 305.1 mm to (352.2, 140.7), turned to 90 degrees
- moved R1 288.3 mm to (305.9, 181.8), turned to 90 degrees
- moved C9 282.7 mm to (337.7, 140.9), turned to 90 degrees
- moved C31 263.0 mm to (311.2, 178.6)
- moved R14 259.6 mm to (312.3, 115.5), turned to -90 degrees
- moved R2 257.9 mm to (273.8, 181.8), turned to 90 degrees
- moved R15 243.8 mm to (295.6, 128.2), turned to 90 degrees
- moved R16 237.3 mm to (289.2, 132.6), turned to 90 degrees
- moved R4 232.4 mm to (245.9, 188.4), turned to 90 degrees
- moved LDR1 229.3 mm to (363.0, 114.0), turned to -90 degrees
- moved R17 224.0 mm to (276.4, 132.8), turned to 90 degrees
- moved R5 217.9 mm to (257.4, 140.0), turned to 90 degrees
- moved C6 216.9 mm to (363.9, 140.8), turned to 90 degrees
- moved C1 214.1 mm to (358.2, 140.7), turned to 90 degrees
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Connections:
- C1 pad 1: Net-(V1A-A) -> Net-(V1B-A)
- C13 pad 1: Net-(V2A-K) -> Net-(V2B-K)
- C14 pad 1: Net-(V1A-K) -> Net-(V1B-K)
- C16 pad 1: Net-(V1B-K) -> Net-(V1A-K)
- C19 pad 2: Net-(V4A-A) -> Net-(V4B-A)
- C2 pad 1: Net-(V1B-A) -> Net-(V1A-A)
- C20 pad 1: Net-(V3B-A) -> Net-(V3A-A)
- C21 pad 1: Net-(V4A-A) -> Net-(V4B-A)
- C22 pad 1: Net-(V3A-A) -> Net-(V3B-A)
- C25 pad 1: Net-(V3A-K) -> Net-(V3B-K)
- C27 pad 1: Net-(V4B-K) -> Net-(V4A-K)
- C28 pad 1: Net-(V3B-K) -> Net-(V3A-K)
- C29 pad 1: Net-(V4A-G) -> Net-(V4B-G)
- C4 pad 1: Net-(V2B-A) -> Net-(V2A-A)
- C5 pad 1: Net-(V2A-A) -> Net-(V2B-A)
- C6 pad 1: Net-(V1A-A) -> Net-(V1B-A)
- R1 pad 2: Net-(V1A-A) -> Net-(V1B-A)
- R11 pad 1: Net-(V2B-K) -> Net-(V2A-K)
- R15 pad 1: Net-(V1A-K) -> Net-(V1B-K)
- R16 pad 1: Net-(V1B-K) -> Net-(V1A-K)
- R2 pad 2: Net-(V1B-A) -> Net-(V1A-A)
- R20 pad 1: Net-(V2A-K) -> Net-(V2B-K)
- R22 pad 1: Net-(V2A-G) -> Net-(V2B-G)
- R24 pad 2: Net-(V3A-A) -> Net-(V3B-A)
- R25 pad 2: Net-(V3B-A) -> Net-(V3A-A)
- R26 pad 2: Net-(V4A-A) -> Net-(V4B-A)
- R29 pad 2: Net-(V4A-G) -> Net-(V4B-G)
- R3 pad 2: Net-(V2B-A) -> Net-(V2A-A)
- R30 pad 2: Net-(V4B-G) -> Net-(V4A-G)
- R31 pad 1: Net-(V4B-G) -> Net-(V4A-G)
- R32 pad 1: Net-(V4B-K) -> Net-(V4A-K)
- R35 pad 1: Net-(V3A-K) -> Net-(V3B-K)
- R37 pad 1: Net-(V3B-G) -> Net-(V3A-G)
- R38 pad 1: Net-(V3B-K) -> Net-(V3A-K)
- R39 pad 1: Net-(V4A-G) -> Net-(V4B-G)
- R4 pad 2: Net-(V2A-A) -> Net-(V2B-A)
- R41 pad 1: Net-(V4A-K) -> Net-(V4B-K)
- R9 pad 1: Net-(V1A-A) -> Net-(V1B-A)
- V1 pad 2: Net-(SW1-A) -> Input
- V1 pad 7: Input -> Net-(SW1-A)
- V2 pad 2: Lead Out -> Net-(V2B-G)
- V2 pad 7: Net-(V2A-G) -> Lead Out
- V3 pad 2: Net-(V3B-G) -> Tank Out
- V3 pad 7: Tank Out -> Net-(V3A-G)
- V4 pad 1: Net-(T1-AB) -> Net-(V4B-A)
- V4 pad 6: Net-(V4A-A) -> Net-(T1-AB)

Commit message: Updated 12AX7 footprint, resized preamp board
Parts:
- V1, V2, V3, V4: footprint Valve:Valve_ECC-83-2 -> IICPP_Clone_Footprints:VT9-ST-C; moved to F.Cu
- moved C10 183.5 mm to (20.6, 64.1)
- moved C12 183.5 mm to (25.5, 71.7)
- moved R12 182.7 mm to (21.5, 78.6)
- moved C19 121.8 mm to (205.0, 90.6)
- moved C29 121.8 mm to (192.5, 81.2)
- moved R26 121.8 mm to (199.6, 93.7)
- moved R30 121.8 mm to (187.5, 92.6)
- moved R31 121.8 mm to (174.9, 88.4)
- moved R25 119.9 mm to (216.9, 89.4)
- moved C21 119.0 mm to (245.7, 56.2)
- moved R27 119.0 mm to (238.5, 36.9)
- moved R38 119.0 mm to (227.7, 49.9)
- moved C28 119.0 mm to (232.8, 51.1)
- moved C20 117.9 mm to (209.7, 78.8)
- moved C24 117.9 mm to (209.5, 54.2)
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Other:
- board outline added: 228.6 x 76.2 mm
- board text added: "HCF Preamp W/ Reverb"
- board text added: "Ver 1.0"

Commit message: initial Preamp Traces
Parts:
- moved C19 195.3 mm to (138.6, 274.2)
- moved D3 195.3 mm to (91.1, 208.8)
- moved R26 195.3 mm to (133.2, 277.3)
- moved R30 195.3 mm to (121.1, 276.2)
- moved C20 195.3 mm to (143.3, 262.4)
- moved C24 195.3 mm to (143.1, 237.8)
- moved C27 195.3 mm to (98.8, 240.3)
- moved C29 195.3 mm to (126.1, 264.8)
- moved C32 195.3 mm to (76.1, 260.1)
- moved D1 195.3 mm to (119.6, 226.9)
- moved D2 195.3 mm to (124.2, 216.7)
- moved D4 195.3 mm to (83.1, 265.1)
- moved D5 195.3 mm to (98.4, 229.0)
- moved LDR4 195.3 mm to (142.7, 212.9)
- moved LDR5 195.3 mm to (94.3, 224.9)
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Routing:
- net Net-(V1C-F1-Pad4): track 0.00 -> 61.0 mm, vias 0 -> 2
- net Net-(V1B-A): track 0.00 -> 57.5 mm
- net Net-(V1B-K): track 0.00 -> 55.3 mm, vias 0 -> 1
- net Net-(V2B-K): track 0.00 -> 47.3 mm
- net E: track 0.00 -> 41.6 mm
- net Net-(C11-Pad1): track 0.00 -> 33.5 mm
- net Net-(C1-Pad2): track 0.00 -> 31.4 mm
- net Net-(V2B-G): track 0.00 -> 28.0 mm
- net Net-(V2B-A): track 0.00 -> 22.1 mm, vias 0 -> 1
- net D: track 0.00 -> 21.2 mm
- net Net-(V2A-A): track 0.00 -> 19.7 mm
- net Net-(C2-Pad2): track 0.00 -> 18.7 mm
- net Net-(V1A-K): track 0.00 -> 17.6 mm
- net Net-(V1A-A): track 0.00 -> 16.9 mm
- net Net-(C6-Pad2): track 0.00 -> 15.0 mm
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
Commit message: Preamp Board Progress
Parts:
- moved LDR4 138.2 mm to (161.2, 76.0)
- moved R29 135.8 mm to (141.8, 109.6)
- moved R39 135.8 mm to (136.5, 124.8)
- moved C20 135.5 mm to (148.8, 127.0)
- moved C19 135.5 mm to (146.6, 139.0)
- moved R26 135.5 mm to (142.1, 142.1)
- moved R25 135.1 mm to (155.2, 138.0)
- moved R6 134.9 mm to (176.0, 134.6)
- moved R37 134.9 mm to (155.2, 113.3)
- moved C24 134.7 mm to (144.9, 103.1)
- moved R41 134.7 mm to (145.1, 97.7)
- moved C29 132.6 mm to (136.5, 132.6)
- moved R27 67.8 mm to (170.4, 77.6)
- moved C22 65.8 mm to (190.8, 116.6)
- moved R42 65.7 mm to (213.8, 94.1)
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Routing:
- net E: track 41.6 -> 159.9 mm
- net Net-(C2-Pad2): track 18.7 -> 109.8 mm, vias 0 -> 1
- net Net-(C23-Pad2): track 0.00 -> 60.4 mm
- net Net-(V4B-A): track 0.00 -> 57.9 mm, vias 0 -> 1
- net Net-(V1C-F2): track 0.00 -> 45.1 mm, vias 0 -> 2
- net Net-(C21-Pad2): track 0.00 -> 41.9 mm
- net Lead Out: track 0.00 -> 41.6 mm
- net D: track 21.2 -> 58.2 mm
- net Net-(V3B-K): track 0.00 -> 33.8 mm
- net Net-(C4-Pad2): track 0.00 -> 32.7 mm, vias 0 -> 1
- net Tank Out: track 0.00 -> 21.3 mm, vias 0 -> 1
- net Net-(V2A-A): track 19.7 -> 35.4 mm
- net Net-(V3B-A): track 0.00 -> 14.0 mm
- net Net-(V4B-G): track 0.00 -> 13.1 mm
- net Net-(V3A-A): track 0.00 -> 11.5 mm
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
Commit message: Preamp board progress, placed most of parts
Parts:
- moved C10 224.2 mm to (243.6, 86.9)
- moved C12 224.2 mm to (248.6, 94.5)
- moved R12 224.2 mm to (244.6, 101.4)
- moved R45 107.7 mm to (146.7, 128.3)
- moved R51 107.4 mm to (174.0, 114.8)
- moved LDR5 107.2 mm to (166.8, 124.7)
- moved R49 106.2 mm to (168.3, 114.8)
- moved D3 106.1 mm to (163.2, 110.3)
- moved C32 98.3 mm to (142.4, 167.4)
- moved D1 97.7 mm to (184.0, 131.8)
- moved D4 97.4 mm to (147.7, 171.1)
- moved D2 96.6 mm to (187.4, 121.7)
- moved R46 94.4 mm to (191.7, 121.7)
- moved D5 88.9 mm to (151.8, 132.2)
- moved C27 88.8 mm to (151.8, 142.8)
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Routing:
- net LDR1+: track 0.00 -> 196.6 mm
- net LDR2-: track 0.00 -> 100.2 mm
- net Net-(D5-K): track 0.00 -> 44.9 mm
- net Net-(C4-Pad2): track 32.7 -> 71.5 mm
- net Reverb In: track 0.00 -> 36.6 mm
- net Net-(LDR5--): track 0.00 -> 27.9 mm
- net Net-(V1C-F1-Pad4): track 61.0 -> 74.8 mm
- net Net-(V4A-K): track 0.00 -> 13.3 mm
- net Net-(V4B-G): track 13.1 -> 20.8 mm
- net Net-(D2-A): track 0.00 -> 6.87 mm
- net Net-(V4B-K): track 0.00 -> 5.48 mm
- net Net-(V4A-G): track 0.00 -> 4.21 mm
Other:
- board size 228.6 x 76.2 mm -> 254 x 76.2 mm
